Commit message: More correct leg positioning

File: hexapod_description/urdf/modules/legs.xacro (robot description, xacro)
@@ -8,8 +8,8 @@
     <xacro:leg index="4" xPos="${-leg1_width/2}" yPos="${body_width/2}" sign="1"/>
     <xacro:leg index="1" xPos="${-leg1_width/2}" yPos="${-body_width/2}" sign="-1"/> -->
-    <xacro:leg index="2" xPos="${body_length/2}" yPos="${body_width/2}" sign="1"/>
-    <xacro:leg index="3" xPos="${body_length/2}" yPos="${-body_width/2}" sign="-1"/>
-    <xacro:leg index="0" xPos="${-body_length/2-leg1_width}" yPos="${body_width/2}" sign="1"/>
-    <xacro:leg index="5" xPos="${-body_length/2-leg1_width}" yPos="${-body_width/2}" sign="-1"/>
+    <xacro:leg index="2" xPos="${body_length/2}" yPos="${front_back_legs_space/2}" sign="1"/>
+    <xacro:leg index="3" xPos="${body_length/2}" yPos="${-front_back_legs_space/2}" sign="-1"/>
+    <xacro:leg index="0" xPos="${-body_length/2-leg1_width}" yPos="${front_back_legs_space/2}" sign="1"/>
+    <xacro:leg index="5" xPos="${-body_length/2-leg1_width}" yPos="${-front_back_legs_space/2}" sign="-1"/>
     <xacro:leg index="1" xPos="${-leg1_width/2}" yPos="${body_width/2}" sign="1"/>
     <xacro:leg index="4" xPos="${-leg1_width/2}" yPos="${-body_width/2}" sign="-1"/>

File: hexapod_description/urdf/modules/robot.xacro (robot description, xacro)
@@ -10,4 +10,5 @@
 	<xacro:property name="body_length" value="0.24"/>
 	<xacro:property name="body_width" value="0.2"/>
+	<xacro:property name="front_back_legs_space" value="0.12"/>
 	<xacro:property name="body_height" value="0.04"/>
 	<xacro:property name="leg1_width" value="0.02"/>

Commit message: Removed unused variables

File: hexapod_description/urdf/modules/legs.xacro (robot description, xacro)
@@ -8,8 +8,8 @@
     <xacro:leg index="4" xPos="${-leg1_width/2}" yPos="${body_width/2}" sign="1"/>
     <xacro:leg index="1" xPos="${-leg1_width/2}" yPos="${-body_width/2}" sign="-1"/> -->
-    <xacro:leg index="2" xPos="${body_length/2-leg1_width/2}" yPos="${front_back_legs_space/2}" sign="1"/>
-    <xacro:leg index="3" xPos="${body_length/2-leg1_width/2}" yPos="${-front_back_legs_space/2}" sign="-1"/>
-    <xacro:leg index="0" xPos="${-body_length/2-leg1_width/2}" yPos="${front_back_legs_space/2}" sign="1"/>
-    <xacro:leg index="5" xPos="${-body_length/2-leg1_width/2}" yPos="${-front_back_legs_space/2}" sign="-1"/>
+    <xacro:leg index="2" xPos="${body_length/2-leg1_width/2}" yPos="${body_length/4}" sign="1"/>
+    <xacro:leg index="3" xPos="${body_length/2-leg1_width/2}" yPos="${-body_length/4}" sign="-1"/>
+    <xacro:leg index="0" xPos="${-body_length/2-leg1_width/2}" yPos="${body_length/4}" sign="1"/>
+    <xacro:leg index="5" xPos="${-body_length/2-leg1_width/2}" yPos="${-body_length/4}" sign="-1"/>
     <xacro:leg index="1" xPos="${-leg1_width/2}" yPos="${body_width/2}" sign="1"/>
     <xacro:leg index="4" xPos="${-leg1_width/2}" yPos="${-body_width/2}" sign="-1"/>

File: hexapod_description/urdf/modules/robot.xacro (robot description, xacro)
@@ -10,5 +10,4 @@
   <xacro:property name="body_length" value="0.24"/>
   <xacro:property name="body_width" value="0.2"/>
-  <xacro:property name="front_back_legs_space" value="0.12"/>
   <xacro:property name="body_height" value="0.04"/>
   <xacro:property name="leg1_width" value="0.02"/>
