Commit message: save, urdf generation not working

File: hexapod_description/urdf/modules/body.xacro (robot description, xacro)
@@ -2,4 +2,10 @@
 <robot xmlns:xacro="http://www.ros.org/wiki/xacro">
     <!-- TORSO -->
+    <link name = "dummy_link"/>
+    <joint name="dummy_link_fix" type="fixed">
+        <parent link="dummy_link"/>
+        <child link="base_link"/>
+        <origin rpy="0 0 -0.3" xyz="-0.14 -0.08 0"/>
+    </joint>
     <link name="base_link">
         <xacro:visuals_collisions_body/>

File: hexapod_description/urdf/modules/leg.xacro (robot description, xacro)
@@ -80,4 +80,15 @@
             </inertial>
         </link>
+        <joint name="sensor_${index}_fix" type="fixed">
+            <parent link="leg_${index}_3"/>
+            <child link="sensor_${index}"/>
+            <origin rpy="0 0 -0.3" xyz="-0.14 -0.08 0"/>
+        </joint>
+        <link name="sensor_${index}"/>
+        <dart_sensor type="force">
+          <link>sensor_${index}</link>
+          <frequency>1000</frequency>
+          <topic>optoforce_${index}</topic>
+        </dart_sensor>
     </xacro:macro>
   <!-- END OF LEG LINKS/JOINTS -->

Commit message: remove dummy link from the body (#9)

File: hexapod_description/urdf/modules/body.xacro (robot description, xacro)
@@ -2,10 +2,4 @@
 <robot xmlns:xacro="http://www.ros.org/wiki/xacro">
     <!-- TORSO -->
-    <link name = "dummy_link"/>
-    <joint name="dummy_link_fix" type="fixed">
-        <parent link="dummy_link"/>
-        <child link="base_link"/>
-        <origin rpy="0 0 -0.3" xyz="-0.14 -0.08 0"/>
-    </joint>
     <link name="base_link">
         <xacro:visuals_collisions_body/>
