Commit message: Romve shifts in x axis in the robot descriptions

File: hexapod_description/urdf/modules/leg_marta.xacro (robot description, xacro)
@@ -8,11 +8,11 @@
             <limit effort="${joint_eff}" lower="${-joint_lim}" upper="${joint_lim}" velocity="${joint_vel}"/>
             <xacro:if value="${index == 5 or index == 2}">
-                <origin rpy="0 0 -0.3" xyz="${xPos} ${yPos-sign*leg1_width} 0"/>
+                <origin rpy="0 0 -0.3" xyz="${xPos} ${yPos} 0"/>
             </xacro:if>
             <xacro:if value="${index == 0 or index == 3}">
-                <origin rpy="0 0 0.3" xyz="${xPos} ${yPos-sign*leg1_width} 0"/>
+                <origin rpy="0 0 0.3" xyz="${xPos} ${yPos} 0"/>
             </xacro:if>
             <xacro:if value="${index == 1 or index == 4}">
-                <origin rpy="0 0 0" xyz="${xPos} ${yPos-sign*leg1_width} 0"/>
+                <origin rpy="0 0 0" xyz="${xPos} ${yPos} 0"/>
             </xacro:if>
             <!-- <xacro:if value="${index == 5 or index == 4 or index == 3}">
@@ -37,5 +37,5 @@
             <parent link="leg_${index}_1"/>
             <child link="leg_${index}_2"/>
-            <limit effort="${joint_eff}" lower="${-joint_lim2}" upper="${joint_lim2}" velocity="${joint_vel}"/>
+            <limit effort="${joint_eff}" lower="${-joint_lim}" upper="${joint_lim}" velocity="${joint_vel}"/>
             <origin rpy="0 0 0" xyz="0 ${sign*leg1_length} 0"/>
             <xacro:if value="${index == 5 or index == 4 or index == 3}">
@@ -60,5 +60,5 @@
             <parent link="leg_${index}_2"/>
             <child link="leg_${index}_3"/>
-            <limit effort="${joint_eff}" lower="${-joint_lim2}" upper="${joint_lim2}" velocity="${joint_vel}"/>
+            <limit effort="${joint_eff}" lower="${-joint_lim}" upper="${joint_lim}" velocity="${joint_vel}"/>
             <origin rpy="${-sign*PI_2} 0 0" xyz="0 ${sign*leg2_length} 0"/>
             <xacro:if value="${index == 5 or index == 4 or index == 3}">
@@ -74,5 +74,5 @@
             <inertial>
                 <!-- CENTER OF MASS -->
-                <origin rpy="${PI_2} 0 0" xyz="${leg3_width/2} ${sign*leg3_length/2} 0"/>
+                <origin rpy="${PI_2} 0 0" xyz="0 ${sign*leg3_length/2} 0"/>
                 <mass value="${leg3_mass}"/>
                 <!-- box inertia: 1/12*m(y^2+z^2), ... -->
@@ -83,5 +83,5 @@
             <parent link="leg_${index}_3"/>
             <child link="force_sensor_${index}"/>
-            <origin rpy="${-sign*PI_2} 0 0" xyz="${leg3_width/2} ${sign*leg3_length} 0"/>
+            <origin rpy="${-sign*PI_2} 0 0" xyz="0 ${sign*leg3_length} ${leg3_dist}"/>
         </joint>
         <link name="force_sensor_${index}"/>

File: hexapod_description/urdf/modules/leg_pexod.xacro (robot description, xacro)
@@ -8,11 +8,11 @@
             <limit effort="${joint_eff}" lower="${-joint_lim}" upper="${joint_lim}" velocity="${joint_vel}"/>
             <xacro:if value="${index == 5 or index == 2}">
-                <origin rpy="0 0 -0.3" xyz="${xPos} ${yPos-sign*leg1_width} 0"/>
+                <origin rpy="0 0 -0.3" xyz="${xPos} ${yPos} 0"/>
             </xacro:if>
             <xacro:if value="${index == 0 or index == 3}">
-                <origin rpy="0 0 0.3" xyz="${xPos} ${yPos-sign*leg1_width} 0"/>
+                <origin rpy="0 0 0.3" xyz="${xPos} ${yPos} 0"/>
             </xacro:if>
             <xacro:if value="${index == 1 or index == 4}">
-                <origin rpy="0 0 0" xyz="${xPos} ${yPos-sign*leg1_width} 0"/>
+                <origin rpy="0 0 0" xyz="${xPos} ${yPos} 0"/>
             </xacro:if>
             <!-- <xacro:if value="${index == 5 or index == 4 or index == 3}">
@@ -74,5 +74,5 @@
             <inertial>
                 <!-- CENTER OF MASS -->
-                <origin rpy="${PI_2} 0 0" xyz="${leg3_width/2} ${sign*leg3_length/2} 0"/>
+                <origin rpy="${PI_2} 0 0" xyz="0 ${sign*leg3_length/2} 0"/>
                 <mass value="${leg3_mass}"/>
                 <!-- box inertia: 1/12*m(y^2+z^2), ... -->

File: hexapod_description/urdf/modules/legs_marta.xacro (robot description, xacro)
@@ -2,10 +2,10 @@
 <robot xmlns:xacro="http://www.ros.org/wiki/xacro">
   <!-- LEGS LINKS/JOINTS -->
-    <xacro:leg index="2" xPos="${body_length/2-leg1_width/2}" yPos="${body_length/4}" sign="1"/>
-    <xacro:leg index="3" xPos="${body_length/2-leg1_width/2}" yPos="${-body_length/4}" sign="-1"/>
-    <xacro:leg index="0" xPos="${-body_length/2-leg1_width/2}" yPos="${body_length/4}" sign="1"/>
-    <xacro:leg index="5" xPos="${-body_length/2-leg1_width/2}" yPos="${-body_length/4}" sign="-1"/>
-    <xacro:leg index="1" xPos="${-leg1_width/2}" yPos="${body_width/2}" sign="1"/>
-    <xacro:leg index="4" xPos="${-leg1_width/2}" yPos="${-body_width/2}" sign="-1"/>
+    <xacro:leg index="2" xPos="${body_length/2}" yPos="${body_width/2}" sign="1"/>
+    <xacro:leg index="3" xPos="${body_length/2}" yPos="${-body_width/2}" sign="-1"/>
+    <xacro:leg index="0" xPos="${-body_length/2}" yPos="${body_width/2}" sign="1"/>
+    <xacro:leg index="5" xPos="${-body_length/2}" yPos="${-body_width/2}" sign="-1"/>
+    <xacro:leg index="1" xPos="0" yPos="${body_width_extra/2}" sign="1"/>
+    <xacro:leg index="4" xPos="0" yPos="${-body_width_extra/2}" sign="-1"/>
   <!-- END OF LEG LINKS/JOINTS -->
 </robot>

File: hexapod_description/urdf/modules/marta.xacro (robot description, xacro)
@@ -8,5 +8,6 @@
   <xacro:property name="body_mass" value="1.031"/>
   <xacro:property name="body_length" value="0.24"/>
-  <xacro:property name="body_width" value="0.2"/>
+  <xacro:property name="body_width" value="0.119"/>
+  <xacro:property name="body_width_extra" value="0.190"/>
   <xacro:property name="body_height" value="0.04"/>
   <xacro:property name="leg1_width" value="0.02"/>
@@ -15,13 +16,12 @@
   <xacro:property name="leg1_mass" value="0.02"/>
   <xacro:property name="leg2_width" value="0.02"/>
-  <xacro:property name="leg2_length" value="0.085"/>
+  <xacro:property name="leg2_length" value="0.0835"/>
   <xacro:property name="leg2_dist" value="0.2"/>
   <xacro:property name="leg2_mass" value="0.184"/>
-  <xacro:property name="leg3_width" value="0.025"/>
-  <xacro:property name="leg3_length" value="0.140"/>
-  <xacro:property name="leg3_dist" value="0.2"/>
+  <xacro:property name="leg3_width" value="0.02"/>
+  <xacro:property name="leg3_length" value="0.12"/>
+  <xacro:property name="leg3_dist" value="0.038"/>
   <xacro:property name="leg3_mass" value="0.04"/>
   <xacro:property name="joint_lim" value="${PI_2}"/>
-  <xacro:property name="joint_lim2" value="${PI_4}"/>
   <xacro:property name="joint_eff" value="30.0"/>
   <xacro:property name="joint_vel" value="7.0"/>

File: hexapod_description/urdf/modules/pexod.xacro (robot description, xacro)
@@ -8,5 +8,6 @@
   <xacro:property name="body_mass" value="1.031"/>
   <xacro:property name="body_length" value="0.24"/>
-  <xacro:property name="body_width" value="0.2"/>
+  <xacro:property name="body_width" value="0.119"/>
+  <xacro:property name="body_width_extra" value="0.190"/>
   <xacro:property name="body_height" value="0.04"/>
   <xacro:property name="leg1_width" value="0.02"/>
@@ -15,10 +16,9 @@
   <xacro:property name="leg1_mass" value="0.02"/>
   <xacro:property name="leg2_width" value="0.02"/>
-  <xacro:property name="leg2_length" value="0.085"/>
+  <xacro:property name="leg2_length" value="0.0835"/>
   <xacro:property name="leg2_dist" value="0.2"/>
   <xacro:property name="leg2_mass" value="0.184"/>
   <xacro:property name="leg3_width" value="0.025"/>
   <xacro:property name="leg3_length" value="0.140"/>
-  <xacro:property name="leg3_dist" value="0.2"/>
   <xacro:property name="leg3_mass" value="0.04"/>
   <xacro:property name="joint_lim" value="${PI_2}"/>
