Commit message: potential error in axis direction

File: hexapod_description/urdf/modules/leg_hexaforce.xacro (robot description, xacro)
@@ -59,5 +59,5 @@
             <limit effort="${joint_eff}" lower="${-joint_lim}" upper="${joint_lim}" velocity="${joint_vel}"/>
             <origin rpy="0 0 0" xyz="0 ${leg2_length} 0"/>
-            <axis xyz="1 0 0"/>
+            <axis xyz="-1 0 0"/>
             <dynamics damping="${joint_dmp}"/>
         </joint>
