Commit message: Minor fix for pexod's leg?

File: hexapod_description/urdf/modules/leg_pexod.xacro (robot description, xacro)
@@ -58,6 +58,6 @@
             <child link="leg_${index}_3"/>
             <limit effort="${joint_eff}" lower="${-joint_lim2}" upper="${joint_lim2}" velocity="${joint_vel}"/>
-            <origin rpy="${PI_2} 0 0" xyz="0 ${leg2_length} 0"/>
-            <axis xyz="1 0 0"/>
+            <origin rpy="0 0 0" xyz="0 ${leg2_length} 0"/>
+            <axis xyz="-1 0 0"/>
             <dynamics damping="${joint_dmp}"/>
         </joint>
