Commit message: fine tune parameters

File: hexapod_description/urdf/modules/hexaforce.xacro (robot description, xacro)
@@ -11,9 +11,9 @@
   <xacro:property name="body_width_extra" value="0.199"/>
   <xacro:property name="body_height" value="0.04"/>
-  <xacro:property name="leg1_width" value="0.05"/>
+  <xacro:property name="leg1_width" value="0.044"/>
   <xacro:property name="leg1_length" value="0.06"/>
   <xacro:property name="leg1_dist" value="0.2"/>
   <xacro:property name="leg1_mass" value="0.02"/>
-  <xacro:property name="leg2_width" value="0.05"/>
+  <xacro:property name="leg2_width" value="0.038"/>
   <xacro:property name="leg2_length" value="0.0835"/>
   <xacro:property name="leg2_dist" value="0.2"/>

Commit message: Add true joint velocities and max torque

File: hexapod_description/urdf/modules/hexaforce.xacro (robot description, xacro)
@@ -27,6 +27,6 @@
   <xacro:property name="force_z_offset" value="0.115"/>
   <xacro:property name="joint_lim" value="${PI_2}"/>
-  <xacro:property name="joint_eff" value="30.0"/>
-  <xacro:property name="joint_vel" value="7.0"/>
+  <xacro:property name="joint_eff" value="2.5"/>
+  <xacro:property name="joint_vel" value="${55*2*PI/60}"/>
   <xacro:property name="joint_dmp" value="0.0"/>
   <xacro:include filename="$(find hexapod_description)/urdf/hexaforce_visuals_collisions.xacro" />

File: hexapod_description/urdf/modules/pexod.xacro (robot description, xacro)
@@ -25,6 +25,6 @@
   <xacro:property name="leg3_mass" value="0.04"/>
   <xacro:property name="joint_lim" value="${PI_2}"/>
-  <xacro:property name="joint_eff" value="30.0"/>
-  <xacro:property name="joint_vel" value="7.0"/>
+  <xacro:property name="joint_eff" value="2.5"/>
+  <xacro:property name="joint_vel" value="${55*2*PI/60}"/>
   <xacro:property name="joint_dmp" value="0.0"/>
   <xacro:include filename="$(find hexapod_description)/urdf/pexod_visuals_collisions.xacro" />

Commit message: Fix for hexaforce empty inertia and adding small damping in joints

File: hexapod_description/urdf/modules/hexaforce.xacro (robot description, xacro)
@@ -29,5 +29,5 @@
   <xacro:property name="joint_eff" value="2.5"/>
   <xacro:property name="joint_vel" value="${55*2*PI/60}"/>
-  <xacro:property name="joint_dmp" value="0.0"/>
+  <xacro:property name="joint_dmp" value="0.1"/>
   <xacro:include filename="$(find hexapod_description)/urdf/hexaforce_visuals_collisions.xacro" />
   <!-- Load xacro modules/parts of the robot -->

File: hexapod_description/urdf/modules/leg_hexaforce.xacro (robot description, xacro)
@@ -77,5 +77,12 @@
             <origin rpy="${PI} 0 ${PI_2}" xyz="0 ${force_y_offset} -${force_z_offset}"/>
         </joint>
-        <link name="force_sensor_${index}"/>
+        <link name="force_sensor_${index}">
+            <!-- Dummy inertia parameters -->
+            <inertial>
+                <origin rpy="0 0 0" xyz="0 0 0"/>
+                <mass value="1e-6"/>
+                <inertia ixx="1e-12" ixy="0" ixz="0" iyy="1e-12" iyz="0" izz="1e-12"/>
+            </inertial>
+        </link>
         <!-- Description used by our Dart simulator -->
         <dart_sensor type="force">

File: hexapod_description/urdf/modules/pexod.xacro (robot description, xacro)
@@ -27,5 +27,5 @@
   <xacro:property name="joint_eff" value="2.5"/>
   <xacro:property name="joint_vel" value="${55*2*PI/60}"/>
-  <xacro:property name="joint_dmp" value="0.0"/>
+  <xacro:property name="joint_dmp" value="0.1"/>
   <xacro:include filename="$(find hexapod_description)/urdf/pexod_visuals_collisions.xacro" />
   <!-- Load xacro modules/parts of the robot -->

Commit message: More realistic joint dynamics

File: hexapod_description/urdf/modules/hexaforce.xacro (robot description, xacro)
@@ -29,5 +29,6 @@
   <xacro:property name="joint_eff" value="2.5"/>
   <xacro:property name="joint_vel" value="${55*2*PI/60}"/>
-  <xacro:property name="joint_dmp" value="0.1"/>
+  <xacro:property name="joint_dmp" value="0.25"/>
+  <xacro:property name="joint_friction" value="0.183333333"/>
   <xacro:include filename="$(find hexapod_description)/urdf/hexaforce_visuals_collisions.xacro" />
   <!-- Load xacro modules/parts of the robot -->

File: hexapod_description/urdf/modules/leg_hexaforce.xacro (robot description, xacro)
@@ -24,5 +24,5 @@
             <origin rpy="0 0 ${offset_angle+legs_rotation}" xyz="${xPos} ${yPos} 0"/>
             <axis xyz="0 0 1"/>
-            <dynamics damping="${joint_dmp}"/>
+            <dynamics damping="${joint_dmp}" friction="${joint_friction}"/>
         </joint>
         <link name="leg_${index}_1">
@@ -42,5 +42,5 @@
             <origin rpy="0 0 0" xyz="0 ${leg1_length} 0"/>
             <axis xyz="1 0 0"/>
-            <dynamics damping="${joint_dmp}"/>
+            <dynamics damping="${joint_dmp}" friction="${joint_friction}"/>
         </joint>
         <link name="leg_${index}_2">
@@ -60,5 +60,5 @@
             <origin rpy="0 0 0" xyz="0 ${leg2_length} 0"/>
             <axis xyz="-1 0 0"/>
-            <dynamics damping="${joint_dmp}"/>
+            <dynamics damping="${joint_dmp}" friction="${joint_friction}"/>
         </joint>
         <link name="leg_${index}_3">

File: hexapod_description/urdf/modules/leg_pexod.xacro (robot description, xacro)
@@ -24,5 +24,5 @@
             <origin rpy="0 0 ${offset_angle+legs_rotation}" xyz="${xPos} ${yPos} 0"/>
             <axis xyz="0 0 1"/>
-            <dynamics damping="${joint_dmp}"/>
+            <dynamics damping="${joint_dmp}" friction="${joint_friction}"/>
         </joint>
         <link name="leg_${index}_1">
@@ -42,5 +42,5 @@
             <origin rpy="0 0 0" xyz="0 ${leg1_length} 0"/>
             <axis xyz="1 0 0"/>
-            <dynamics damping="${joint_dmp}"/>
+            <dynamics damping="${joint_dmp}" friction="${joint_friction}"/>
         </joint>
         <link name="leg_${index}_2">
@@ -60,5 +60,5 @@
             <origin rpy="0 0 0" xyz="0 ${leg2_length} 0"/>
             <axis xyz="-1 0 0"/>
-            <dynamics damping="${joint_dmp}"/>
+            <dynamics damping="${joint_dmp}" friction="${joint_friction}"/>
         </joint>
         <link name="leg_${index}_3">

File: hexapod_description/urdf/modules/pexod.xacro (robot description, xacro)
@@ -27,5 +27,6 @@
   <xacro:property name="joint_eff" value="2.5"/>
   <xacro:property name="joint_vel" value="${55*2*PI/60}"/>
-  <xacro:property name="joint_dmp" value="0.1"/>
+  <xacro:property name="joint_dmp" value="0.25"/>
+  <xacro:property name="joint_friction" value="0.183333333"/>
   <xacro:include filename="$(find hexapod_description)/urdf/pexod_visuals_collisions.xacro" />
   <!-- Load xacro modules/parts of the robot -->
