Commit message: Parameters for mini-hexapod xacro update

File: hexapod_description/urdf/modules/mini_hexapod.xacro (robot description, xacro)
@@ -6,22 +6,22 @@
   <xacro:property name="PI_4" value="0.78539816339" />
   <xacro:property name="scale" value="0.001" />
-  <xacro:property name="body_mass" value="1.031"/>
-  <xacro:property name="body_length" value="0.24"/>
-  <xacro:property name="body_width" value="0.119"/>
-  <xacro:property name="body_width_extra" value="0.199"/>
-  <xacro:property name="body_height" value="0.04"/>
-  <xacro:property name="leg1_width" value="0.044"/>
-  <xacro:property name="leg1_length" value="0.06"/>
+  <xacro:property name="body_mass" value="0.322"/>
+  <xacro:property name="body_length" value="0.145"/>
+  <xacro:property name="body_width" value="0.095"/>
+  <xacro:property name="body_width_extra" value="0.095"/>
+  <xacro:property name="body_height" value="0.035"/>
+  <xacro:property name="leg1_width" value="0.0345"/>
+  <xacro:property name="leg1_length" value="0.047"/>
   <xacro:property name="leg1_dist" value="0.2"/>
-  <xacro:property name="leg1_mass" value="0.02"/>
-  <xacro:property name="leg2_width" value="0.038"/>
-  <xacro:property name="leg2_length" value="0.0835"/>
+  <xacro:property name="leg1_mass" value="0.01141"/>
+  <xacro:property name="leg2_width" value="0.034"/>
+  <xacro:property name="leg2_length" value="0.06"/>
   <xacro:property name="leg2_dist" value="0.2"/>
-  <xacro:property name="leg2_mass" value="0.184"/>
-  <xacro:property name="leg3_width" value="0.054"/>
-  <xacro:property name="leg3_length" value="0.065"/>
+  <xacro:property name="leg2_mass" value="0.04272"/>
+  <xacro:property name="leg3_width" value="0.0345"/>
+  <xacro:property name="leg3_length" value="0.01"/>
   <xacro:property name="leg3_height" value="0.10"/>
   <xacro:property name="leg3_tip_radius" value="0.02"/>
-  <xacro:property name="leg3_mass" value="0.04"/>
+  <xacro:property name="leg3_mass" value="0.01457"/>
   <xacro:property name="joint_lim" value="${PI_2}"/>
   <xacro:property name="joint_eff" value="2.5"/>
