Commit message: First working version on real robot

File: hexapod_description/urdf/modules/leg.xacro (robot description, xacro)
@@ -20,5 +20,5 @@
             </xacro:if>
             <xacro:if value="${index == 2 or index == 1 or index == 0}"> -->
-                <axis xyz="0 0 -1"/>
+                <axis xyz="0 0 1"/>
             <!-- </xacro:if> -->
             <dynamics damping="${joint_dmp}"/>
@@ -40,8 +40,8 @@
             <origin rpy="0 0 0" xyz="0 ${sign*leg1_length} 0"/>
             <xacro:if value="${index == 5 or index == 4 or index == 3}">
-                <axis xyz="1 0 0"/>
+                <axis xyz="-1 0 0"/>
             </xacro:if>
             <xacro:if value="${index == 2 or index == 1 or index == 0}">
-                <axis xyz="-1 0 0"/>
+                <axis xyz="1 0 0"/>
             </xacro:if>
             <dynamics damping="${joint_dmp}"/>

Commit message: Removed all tabs

File: hexapod_description/urdf/modules/leg.xacro (robot description, xacro)
@@ -1,5 +1,5 @@
 <?xml version="1.0"?>
 <robot xmlns:xacro="http://www.ros.org/wiki/xacro">
-	<!-- XACRO MACRO FOR LEGS LINKS/JOINTS -->
+  <!-- XACRO MACRO FOR LEGS LINKS/JOINTS -->
     <xacro:macro name="leg" params="index xPos yPos sign">
         <joint name="body_leg_${index}" type="revolute">
@@ -81,4 +81,4 @@
         </link>
     </xacro:macro>
-    <!-- END OF LEG LINKS/JOINTS -->
+  <!-- END OF LEG LINKS/JOINTS -->
 </robot>

File: hexapod_description/urdf/modules/legs.xacro (robot description, xacro)
@@ -1,5 +1,5 @@
 <?xml version="1.0"?>
 <robot xmlns:xacro="http://www.ros.org/wiki/xacro">
-	<!-- LEGS LINKS/JOINTS -->
+  <!-- LEGS LINKS/JOINTS -->
     <!-- <xacro:leg index="5" xPos="${body_length/2}" yPos="${body_width/2}" sign="1"/>
     <xacro:leg index="0" xPos="${body_length/2}" yPos="${-body_width/2}" sign="-1"/>
@@ -14,4 +14,4 @@
     <xacro:leg index="1" xPos="${-leg1_width/2}" yPos="${body_width/2}" sign="1"/>
     <xacro:leg index="4" xPos="${-leg1_width/2}" yPos="${-body_width/2}" sign="-1"/>
-    <!-- END OF LEG LINKS/JOINTS -->
+  <!-- END OF LEG LINKS/JOINTS -->
 </robot>

File: hexapod_description/urdf/modules/robot.xacro (robot description, xacro)
@@ -1,41 +1,41 @@
 <?xml version="1.0"?>
 <robot xmlns:xacro="http://www.ros.org/wiki/xacro">
-	<!-- XACRO PROPERTIES -->
-	<xacro:property name="PI" value="3.14159265359" />
-	<xacro:property name="PI_2" value="1.57079632679" />
-	<xacro:property name="PI_4" value="0.78539816339" />
-	<xacro:property name="scale" value="0.001" />
-	<xacro:property name="use_gazebo" value="true" />
-	<xacro:property name="body_mass" value="1.031"/>
-	<xacro:property name="body_length" value="0.24"/>
-	<xacro:property name="body_width" value="0.2"/>
-	<xacro:property name="front_back_legs_space" value="0.12"/>
-	<xacro:property name="body_height" value="0.04"/>
-	<xacro:property name="leg1_width" value="0.02"/>
-	<xacro:property name="leg1_length" value="0.06"/>
-	<xacro:property name="leg1_dist" value="0.2"/>
-	<xacro:property name="leg1_mass" value="0.02"/>
-	<xacro:property name="leg2_width" value="0.02"/>
-	<xacro:property name="leg2_length" value="0.085"/>
-	<xacro:property name="leg2_dist" value="0.2"/>
-	<xacro:property name="leg2_mass" value="0.184"/>
-	<xacro:property name="leg3_width" value="0.025"/>
-	<xacro:property name="leg3_length" value="0.140"/>
-	<xacro:property name="leg3_dist" value="0.2"/>
-	<xacro:property name="leg3_mass" value="0.04"/>
-	<xacro:property name="joint_lim" value="${PI_2}"/>
-	<xacro:property name="joint_lim2" value="${PI_4}"/>
-	<xacro:property name="joint_eff" value="30.0"/>
-	<xacro:property name="joint_vel" value="7.0"/>
-	<xacro:property name="joint_dmp" value="0.0"/>
-	<xacro:include filename="$(find hexapod_description)/urdf/pexod_visuals_collisions.xacro" />
-	<xacro:if value="${use_gazebo}">
-		<!-- <xacro:include filename="$(find hexapod_description)/urdf/pexod_gazebo.xacro" /> -->
-	</xacro:if>
-	<!-- Load xacro modules/parts of the robot -->
-	<xacro:include filename="$(find hexapod_description)/urdf/modules/body.xacro" />
-	<xacro:include filename="$(find hexapod_description)/urdf/modules/leg.xacro" />
-	<xacro:include filename="$(find hexapod_description)/urdf/modules/legs.xacro" />
-	<!-- <xacro:include filename="$(find hexapod_description)/urdf/modules/imu.xacro" /> -->
-	<!-- <xacro:include filename="$(find hexapod_description)/urdf/modules/cameras.xacro" /> -->
+  <!-- XACRO PROPERTIES -->
+  <xacro:property name="PI" value="3.14159265359" />
+  <xacro:property name="PI_2" value="1.57079632679" />
+  <xacro:property name="PI_4" value="0.78539816339" />
+  <xacro:property name="scale" value="0.001" />
+  <xacro:property name="use_gazebo" value="true" />
+  <xacro:property name="body_mass" value="1.031"/>
+  <xacro:property name="body_length" value="0.24"/>
+  <xacro:property name="body_width" value="0.2"/>
+  <xacro:property name="front_back_legs_space" value="0.12"/>
+  <xacro:property name="body_height" value="0.04"/>
+  <xacro:property name="leg1_width" value="0.02"/>
+  <xacro:property name="leg1_length" value="0.06"/>
+  <xacro:property name="leg1_dist" value="0.2"/>
+  <xacro:property name="leg1_mass" value="0.02"/>
+  <xacro:property name="leg2_width" value="0.02"/>
+  <xacro:property name="leg2_length" value="0.085"/>
+  <xacro:property name="leg2_dist" value="0.2"/>
+  <xacro:property name="leg2_mass" value="0.184"/>
+  <xacro:property name="leg3_width" value="0.025"/>
+  <xacro:property name="leg3_length" value="0.140"/>
+  <xacro:property name="leg3_dist" value="0.2"/>
+  <xacro:property name="leg3_mass" value="0.04"/>
+  <xacro:property name="joint_lim" value="${PI_2}"/>
+  <xacro:property name="joint_lim2" value="${PI_4}"/>
+  <xacro:property name="joint_eff" value="30.0"/>
+  <xacro:property name="joint_vel" value="7.0"/>
+  <xacro:property name="joint_dmp" value="0.0"/>
+  <xacro:include filename="$(find hexapod_description)/urdf/pexod_visuals_collisions.xacro" />
+  <xacro:if value="${use_gazebo}">
+    <!-- <xacro:include filename="$(find hexapod_description)/urdf/pexod_gazebo.xacro" /> -->
+  </xacro:if>
+  <!-- Load xacro modules/parts of the robot -->
+  <xacro:include filename="$(find hexapod_description)/urdf/modules/body.xacro" />
+  <xacro:include filename="$(find hexapod_description)/urdf/modules/leg.xacro" />
+  <xacro:include filename="$(find hexapod_description)/urdf/modules/legs.xacro" />
+  <!-- <xacro:include filename="$(find hexapod_description)/urdf/modules/imu.xacro" /> -->
+  <!-- <xacro:include filename="$(find hexapod_description)/urdf/modules/cameras.xacro" /> -->
 </robot>

File: hexapod_description/urdf/pexod.xacro (robot description, xacro)
@@ -1,5 +1,5 @@
 <?xml version="1.0"?>
 <robot name="pexod" xmlns:xacro="http://www.ros.org/wiki/xacro">
-	<!-- <xacro:include filename="$(find pexod_description)/urdf/pexod_control.xacro" /> -->
-	<xacro:include filename="$(find hexapod_description)/urdf/modules/robot.xacro" />
+  <!-- <xacro:include filename="$(find pexod_description)/urdf/pexod_control.xacro" /> -->
+  <xacro:include filename="$(find hexapod_description)/urdf/modules/robot.xacro" />
 </robot>

File: hexapod_description/urdf/pexod_visuals_collisions.xacro (robot description, xacro)
@@ -1,96 +1,96 @@
 <?xml version="1.0"?>
 <robot xmlns:xacro="http://www.ros.org/wiki/xacro">
-	<!-- MATERIALS -->
-	<material name="Blue">
-		<color rgba="0 0 1 1"/>
+  <!-- MATERIALS -->
+  <material name="Blue">
+    <color rgba="0 0 1 1"/>
     </material>
     <material name="Red">
-    	<color rgba="1 0 0 1"/>
-  	</material>
-  	<material name="Green">
+      <color rgba="1 0 0 1"/>
+    </material>
+    <material name="Green">
         <color rgba="0 1 0 1"/>
-	</material>
-	<material name="Yellow">
-		<color rgba="1 1 0 1"/>
+  </material>
+  <material name="Yellow">
+    <color rgba="1 1 0 1"/>
     </material>
     <material name="LightGrey">
-    	<color rgba="0.6 0.6 0.6 1.0"/>
-	</material>
+      <color rgba="0.6 0.6 0.6 1.0"/>
+  </material>
     <!-- END OF MATERIALS -->
     <!-- XACRO MACROS FOR VISUALS AND COLLISIONS -->
     <xacro:macro name="visuals_collisions_body" params="">
-		<visual>
-			<origin xyz="0 0 0" rpy="0 0 0"/>
+    <visual>
+      <origin xyz="0 0 0" rpy="0 0 0"/>
             <geometry>
                 <box size="${body_length} ${body_width} ${body_height}"/>
             </geometry>
-			<material name="Blue"/>
-		</visual>
-		<collision>
-			<origin xyz="0 0 0" rpy="0 0 0"/>
+      <material name="Blue"/>
+    </visual>
+    <collision>
+      <origin xyz="0 0 0" rpy="0 0 0"/>
             <geometry>
                 <box size="${body_length} ${body_width} ${body_height}"/>
             </geometry>
-		</collision>
-	</xacro:macro>
-	<xacro:macro name="visuals_collisions_leg_1" params="revert">
-		<visual>
-			<origin xyz="${leg1_width/2} ${revert*leg1_length/2} 0" rpy="${PI_2} 0 0"/>
+    </collision>
+  </xacro:macro>
+  <xacro:macro name="visuals_collisions_leg_1" params="revert">
+    <visual>
+      <origin xyz="${leg1_width/2} ${revert*leg1_length/2} 0" rpy="${PI_2} 0 0"/>
             <geometry>
                 <cylinder radius="${leg1_width}" length="${leg1_length}"/>
             </geometry>
-			<material name="Red"/>
-		</visual>
-		<collision>
-			<origin xyz="${leg1_width/2} ${revert*leg1_length/2} 0" rpy="${PI_2} 0 0"/>
+      <material name="Red"/>
+    </visual>
+    <collision>
+      <origin xyz="${leg1_width/2} ${revert*leg1_length/2} 0" rpy="${PI_2} 0 0"/>
             <geometry>
                 <box size="${1.5*leg1_width} ${1.5*leg1_width} ${leg1_length}"/>
             </geometry>
-		</collision>
-	</xacro:macro>
-	<xacro:macro name="visuals_collisions_leg_2" params="revert">
-		<visual>
-			<origin xyz="${leg2_width/2} ${revert*leg2_length/2} 0" rpy="${PI_2} 0 0"/>
+    </collision>
+  </xacro:macro>
+  <xacro:macro name="visuals_collisions_leg_2" params="revert">
+    <visual>
+      <origin xyz="${leg2_width/2} ${revert*leg2_length/2} 0" rpy="${PI_2} 0 0"/>
             <geometry>
                 <cylinder radius="${leg2_width}" length="${leg2_length}"/>
             </geometry>
-			<material name="Blue"/>
-		</visual>
-		<collision>
-			<origin xyz="${leg2_width/2} ${revert*leg2_length/2} 0" rpy="${PI_2} 0 0"/>
+      <material name="Blue"/>
+    </visual>
+    <collision>
+      <origin xyz="${leg2_width/2} ${revert*leg2_length/2} 0" rpy="${PI_2} 0 0"/>
             <geometry>
                 <box size="${1.5*leg2_width} ${1.5*leg2_width} ${leg2_length}"/>
             </geometry>
-		</collision>
-	</xacro:macro>
-	<xacro:macro name="visuals_collisions_leg_3" params="revert">
-		<visual>
-			<origin xyz="${leg3_width/2} ${revert*leg3_length/2} 0" rpy="${PI_2} 0 0"/>
+    </collision>
+  </xacro:macro>
+  <xacro:macro name="visuals_collisions_leg_3" params="revert">
+    <visual>
+      <origin xyz="${leg3_width/2} ${revert*leg3_length/2} 0" rpy="${PI_2} 0 0"/>
             <geometry>
               <cylinder radius="${leg3_width}" length="${leg3_length}"/>
             </geometry>
-			<material name="Red"/>
-		</visual>
-		<visual>
-			<origin xyz="${leg3_width/2} ${revert*leg3_length-revert*leg3_width/2} 0" rpy="${PI_2} 0 0"/>
+      <material name="Red"/>
+    </visual>
+    <visual>
+      <origin xyz="${leg3_width/2} ${revert*leg3_length-revert*leg3_width/2} 0" rpy="${PI_2} 0 0"/>
             <geometry>
                 <sphere radius="${leg3_width}"/>
             </geometry>
-			<material name="Red"/>
-		</visual>
-		<collision>
-			<origin xyz="${leg3_width/2} ${revert*leg3_length/2} 0" rpy="${PI_2} 0 0"/>
+      <material name="Red"/>
+    </visual>
+    <collision>
+      <origin xyz="${leg3_width/2} ${revert*leg3_length/2} 0" rpy="${PI_2} 0 0"/>
             <geometry>
                 <box size="${1.5*leg3_width} ${1.5*leg3_width} ${leg3_length}"/>
             </geometry>
-		</collision>
-		<collision>
-			<origin xyz="${leg3_width/2} ${revert*leg3_length-revert*leg3_width/2} 0" rpy="${PI_2} 0 0"/>
+    </collision>
+    <collision>
+      <origin xyz="${leg3_width/2} ${revert*leg3_length-revert*leg3_width/2} 0" rpy="${PI_2} 0 0"/>
             <geometry>
                 <sphere radius="${leg3_width}"/>
             </geometry>
-			<material name="Red"/>
-		</collision>
-	</xacro:macro>
-	<!-- END OF XACRO MACROS -->
+      <material name="Red"/>
+    </collision>
+  </xacro:macro>
+  <!-- END OF XACRO MACROS -->
 </robot>

Commit message: Fixed inertia properties + fix in collision shapes

File: hexapod_description/urdf/modules/leg.xacro (robot description, xacro)
@@ -30,6 +30,6 @@
                 <origin rpy="${PI_2} 0 0" xyz="${leg1_width/2} ${sign*leg1_length/2} 0"/>
                 <mass value="${leg1_mass}"/>
-                <!-- Cylinder inertia: 1/12*m*(3*r^2+h^2), 1/12*m*(3*r^2+h^2), 1/12*m*r^2 -->
-                <inertia ixx="${1/12*leg1_mass*(3*leg1_width*leg1_width+leg1_length*leg1_length)}" ixy="0" ixz="0" iyy="${1/12*leg1_mass*(3*leg1_width*leg1_width+leg1_length*leg1_length)}" iyz="0" izz="${1/12*leg1_mass*leg1_width*leg1_width}"/>
+                <!-- box inertia: 1/12*m(y^2+z^2), ... -->
+                <inertia ixx="${1/12*leg1_mass*(leg1_width*leg1_width+leg1_length*leg1_length)}" ixy="0" ixz="0" iyy="${1/12*leg1_mass*(leg1_width*leg1_width+leg1_length*leg1_length)}" iyz="0" izz="${1/12*leg1_mass*(2*leg1_width*leg1_width)}"/>
             </inertial>
         </link>
@@ -53,6 +53,6 @@
                 <origin rpy="${PI_2} 0 0" xyz="${leg2_width/2} ${sign*leg2_length/2} 0"/>
                 <mass value="${leg2_mass}"/>
-                <!-- Cylinder inertia: 1/12*m*(3*r^2+h^2), 1/12*m*(3*r^2+h^2), 1/12*m*r^2 -->
-                <inertia ixx="${1/12*leg2_mass*(3*leg2_width*leg2_width+leg2_length*leg2_length)}" ixy="0" ixz="0" iyy="${1/12*leg2_mass*(3*leg2_width*leg2_width+leg2_length*leg2_length)}" iyz="0" izz="${1/12*leg2_mass*leg2_width*leg2_width}"/>
+                <!-- box inertia: 1/12*m(y^2+z^2), ... -->
+                <inertia ixx="${1/12*leg2_mass*(leg2_width*leg2_width+leg2_length*leg2_length)}" ixy="0" ixz="0" iyy="${1/12*leg2_mass*(leg2_width*leg2_width+leg2_length*leg2_length)}" iyz="0" izz="${1/12*leg2_mass*(2*leg2_width*leg2_width)}"/>
             </inertial>
         </link>
@@ -75,7 +75,7 @@
                 <!-- CENTER OF MASS -->
                 <origin rpy="${PI_2} 0 0" xyz="${leg3_width/2} ${sign*leg3_length/2} 0"/>
-                <mass value="${leg2_mass}"/>
-                <!-- Cylinder inertia: 1/12*m*(3*r^2+h^2), 1/12*m*(3*r^2+h^2), 1/12*m*r^2 -->
-                <inertia ixx="${1/12*leg2_mass*(3*leg2_width*leg2_width+leg2_length*leg2_length)}" ixy="0" ixz="0" iyy="${1/12*leg2_mass*(3*leg2_width*leg2_width+leg2_length*leg2_length)}" iyz="0" izz="${1/12*leg2_mass*leg2_width*leg2_width}"/>
+                <mass value="${leg3_mass}"/>
+                <!-- box inertia: 1/12*m(y^2+z^2), ... -->
+                <inertia ixx="${1/12*leg3_mass*(leg3_width*leg3_width+leg3_length*leg3_length)}" ixy="0" ixz="0" iyy="${1/12*leg3_mass*(leg3_width*leg3_width+leg3_length*leg3_length)}" iyz="0" izz="${1/12*leg3_mass*(2*leg3_width*leg3_width)}"/>
             </inertial>
         </link>

File: hexapod_description/urdf/pexod_visuals_collisions.xacro (robot description, xacro)
@@ -45,5 +45,5 @@
       <origin xyz="${leg1_width/2} ${revert*leg1_length/2} 0" rpy="${PI_2} 0 0"/>
             <geometry>
-                <box size="${1.5*leg1_width} ${1.5*leg1_width} ${leg1_length}"/>
+                <box size="${leg1_width} ${leg1_width} ${leg1_length}"/>
             </geometry>
     </collision>
@@ -60,5 +60,5 @@
       <origin xyz="${leg2_width/2} ${revert*leg2_length/2} 0" rpy="${PI_2} 0 0"/>
             <geometry>
-                <box size="${1.5*leg2_width} ${1.5*leg2_width} ${leg2_length}"/>
+                <box size="${leg2_width} ${leg2_width} ${leg2_length}"/>
             </geometry>
     </collision>
@@ -82,5 +82,5 @@
       <origin xyz="${leg3_width/2} ${revert*leg3_length/2} 0" rpy="${PI_2} 0 0"/>
             <geometry>
-                <box size="${1.5*leg3_width} ${1.5*leg3_width} ${leg3_length}"/>
+                <box size="${leg3_width} ${leg3_width} ${leg3_length}"/>
             </geometry>
     </collision>

Commit message: corrected sensorsposition

File: hexapod_description/urdf/modules/leg.xacro (robot description, xacro)
@@ -83,5 +83,5 @@
             <parent link="leg_${index}_3"/>
             <child link="sensor_${index}"/>
-            <origin rpy="0 0 -0.3" xyz="-0.14 -0.08 0"/>
+            <origin rpy="${-sign*PI_2} 0 0" xyz="${leg3_width/2} ${sign*leg3_length} 0"/>
         </joint>
         <link name="sensor_${index}"/>

Commit message: added transmissions

File: hexapod_description/urdf/modules/leg.xacro (robot description, xacro)
@@ -91,4 +91,34 @@
           <topic>optoforce_${index}</topic>
         </dart_sensor>
+        <transmission name="tran${index}1">
+            <type>transmission_interface/SimpleTransmission</type>
+            <joint name="body_leg_${index}">
+                <hardwareInterface>PositionJointInterface</hardwareInterface>
+            </joint>
+            <actuator name="motor${index}1">
+                <hardwareInterface>PositionJointInterface</hardwareInterface>
+                <mechanicalReduction>1</mechanicalReduction>
+            </actuator>
+        </transmission>
+        <transmission name="tran${index}2">
+            <type>transmission_interface/SimpleTransmission</type>
+            <joint name="leg_${index}_1_2">
+                <hardwareInterface>PositionJointInterface</hardwareInterface>
+            </joint>
+            <actuator name="motor${index}2">
+                <hardwareInterface>PositionJointInterface</hardwareInterface>
+                <mechanicalReduction>1</mechanicalReduction>
+            </actuator>
+        </transmission>
+        <transmission name="tran${index}3">
+            <type>transmission_interface/SimpleTransmission</type>
+            <joint name="leg_${index}_2_3">
+                <hardwareInterface>PositionJointInterface</hardwareInterface>
+            </joint>
+            <actuator name="motor${index}2">
+                <hardwareInterface>PositionJointInterface</hardwareInterface>
+                <mechanicalReduction>1</mechanicalReduction>
+            </actuator>
+        </transmission>
     </xacro:macro>
   <!-- END OF LEG LINKS/JOINTS -->

Commit message: update sensor frames in URDF

File: hexapod_description/urdf/modules/leg.xacro (robot description, xacro)
@@ -2,5 +2,5 @@
 <robot xmlns:xacro="http://www.ros.org/wiki/xacro">
   <!-- XACRO MACRO FOR LEGS LINKS/JOINTS -->
-    <xacro:macro name="leg" params="index xPos yPos sign">
+    <xacro:macro name="leg" params="index xPos yPos sign serial_number">
         <joint name="body_leg_${index}" type="revolute">
             <parent link="base_link"/>
@@ -80,12 +80,12 @@
             </inertial>
         </link>
-        <joint name="sensor_${index}_fix" type="fixed">
+        <joint name="optoforce_${serial_number}_0_fix" type="fixed">
             <parent link="leg_${index}_3"/>
-            <child link="sensor_${index}"/>
+            <child link="optoforce_${serial_number}_0"/>
             <origin rpy="${-sign*PI_2} 0 0" xyz="${leg3_width/2} ${sign*leg3_length} 0"/>
         </joint>
-        <link name="sensor_${index}"/>
+        <link name="optoforce_${serial_number}_0"/>
         <dart_sensor type="force">
-          <link>sensor_${index}</link>
+          <link>optoforce_${serial_number}_0</link>
           <frequency>1000</frequency>
           <topic>optoforce_${index}</topic>

File: hexapod_description/urdf/modules/legs.xacro (robot description, xacro)
@@ -8,10 +8,10 @@
     <xacro:leg index="4" xPos="${-leg1_width/2}" yPos="${body_width/2}" sign="1"/>
     <xacro:leg index="1" xPos="${-leg1_width/2}" yPos="${-body_width/2}" sign="-1"/> -->
-    <xacro:leg index="2" xPos="${body_length/2-leg1_width/2}" yPos="${body_length/4}" sign="1"/>
-    <xacro:leg index="3" xPos="${body_length/2-leg1_width/2}" yPos="${-body_length/4}" sign="-1"/>
-    <xacro:leg index="0" xPos="${-body_length/2-leg1_width/2}" yPos="${body_length/4}" sign="1"/>
-    <xacro:leg index="5" xPos="${-body_length/2-leg1_width/2}" yPos="${-body_length/4}" sign="-1"/>
-    <xacro:leg index="1" xPos="${-leg1_width/2}" yPos="${body_width/2}" sign="1"/>
-    <xacro:leg index="4" xPos="${-leg1_width/2}" yPos="${-body_width/2}" sign="-1"/>
+    <xacro:leg index="2" serial_number="ISE175" xPos="${body_length/2-leg1_width/2}" yPos="${body_length/4}" sign="1"/>
+    <xacro:leg index="3" serial_number="ISE177" xPos="${body_length/2-leg1_width/2}" yPos="${-body_length/4}" sign="-1"/>
+    <xacro:leg index="0" serial_number="ISE182" xPos="${-body_length/2-leg1_width/2}" yPos="${body_length/4}" sign="1"/>
+    <xacro:leg index="5" serial_number="ISE173" xPos="${-body_length/2-leg1_width/2}" yPos="${-body_length/4}" sign="-1"/>
+    <xacro:leg index="1" serial_number="ISE174" xPos="${-leg1_width/2}" yPos="${body_width/2}" sign="1"/>
+    <xacro:leg index="4" serial_number="ISE184" xPos="${-leg1_width/2}" yPos="${-body_width/2}" sign="-1"/>
   <!-- END OF LEG LINKS/JOINTS -->
 </robot>
