Commit message: reverting to generic names for sensor frames

File: hexapod_description/urdf/modules/leg.xacro (robot description, xacro)
@@ -2,5 +2,5 @@
 <robot xmlns:xacro="http://www.ros.org/wiki/xacro">
   <!-- XACRO MACRO FOR LEGS LINKS/JOINTS -->
-    <xacro:macro name="leg" params="index xPos yPos sign serial_number">
+    <xacro:macro name="leg" params="index xPos yPos sign">
         <joint name="body_leg_${index}" type="revolute">
             <parent link="base_link"/>
@@ -80,12 +80,12 @@
             </inertial>
         </link>
-        <joint name="optoforce_${serial_number}_0_fix" type="fixed">
+        <joint name="force_sensor_${index}_fix" type="fixed">
             <parent link="leg_${index}_3"/>
-            <child link="optoforce_${serial_number}_0"/>
+            <child link="force_sensor_${index}"/>
             <origin rpy="${-sign*PI_2} 0 0" xyz="${leg3_width/2} ${sign*leg3_length} 0"/>
         </joint>
-        <link name="optoforce_${serial_number}_0"/>
+        <link name="force_sensor_${index}"/>
         <dart_sensor type="force">
-          <link>optoforce_${serial_number}_0</link>
+          <link>force_sensor_${index}</link>
           <frequency>1000</frequency>
           <topic>optoforce_${index}</topic>

File: hexapod_description/urdf/modules/legs.xacro (robot description, xacro)
@@ -2,10 +2,10 @@
 <robot xmlns:xacro="http://www.ros.org/wiki/xacro">
   <!-- LEGS LINKS/JOINTS -->
-    <xacro:leg index="2" serial_number="ISE174" xPos="${body_length/2-leg1_width/2}" yPos="${body_length/4}" sign="1"/>
-    <xacro:leg index="3" serial_number="ISE184" xPos="${body_length/2-leg1_width/2}" yPos="${-body_length/4}" sign="-1"/>
-    <xacro:leg index="0" serial_number="ISE175" xPos="${-body_length/2-leg1_width/2}" yPos="${body_length/4}" sign="1"/>
-    <xacro:leg index="5" serial_number="ISE177" xPos="${-body_length/2-leg1_width/2}" yPos="${-body_length/4}" sign="-1"/>
-    <xacro:leg index="1" serial_number="ISE173" xPos="${-leg1_width/2}" yPos="${body_width/2}" sign="1"/>
-    <xacro:leg index="4" serial_number="ISE182" xPos="${-leg1_width/2}" yPos="${-body_width/2}" sign="-1"/>
+    <xacro:leg index="2" xPos="${body_length/2-leg1_width/2}" yPos="${body_length/4}" sign="1"/>
+    <xacro:leg index="3" xPos="${body_length/2-leg1_width/2}" yPos="${-body_length/4}" sign="-1"/>
+    <xacro:leg index="0" xPos="${-body_length/2-leg1_width/2}" yPos="${body_length/4}" sign="1"/>
+    <xacro:leg index="5" xPos="${-body_length/2-leg1_width/2}" yPos="${-body_length/4}" sign="-1"/>
+    <xacro:leg index="1" xPos="${-leg1_width/2}" yPos="${body_width/2}" sign="1"/>
+    <xacro:leg index="4" xPos="${-leg1_width/2}" yPos="${-body_width/2}" sign="-1"/>
   <!-- END OF LEG LINKS/JOINTS -->
 </robot>

Commit message: remove force sensors from Pexod's Xacro description

File: hexapod_description/urdf/modules/leg.xacro (robot description, xacro)
@@ -80,15 +80,4 @@
             </inertial>
         </link>
-        <joint name="force_sensor_${index}_fix" type="fixed">
-            <parent link="leg_${index}_3"/>
-            <child link="force_sensor_${index}"/>
-            <origin rpy="${-sign*PI_2} 0 0" xyz="${leg3_width/2} ${sign*leg3_length} 0"/>
-        </joint>
-        <link name="force_sensor_${index}"/>
-        <dart_sensor type="force">
-          <link>force_sensor_${index}</link>
-          <frequency>1000</frequency>
-          <topic>optoforce_${index}</topic>
-        </dart_sensor>
         <transmission name="tran${index}1">
             <type>transmission_interface/SimpleTransmission</type>

Commit message: Saving files for backup -- to inspect

File: hexapod_description/urdf/modules/leg.xacro (robot description, xacro)
@@ -71,5 +71,5 @@
         </joint>
         <link name="leg_${index}_3">
-            <xacro:visuals_collisions_leg_3 revert="${sign}"/>
+            <xacro:visuals_collisions_leg_3 revert="${sign}" index="${index}"/>
             <inertial>
                 <!-- CENTER OF MASS -->

File: hexapod_description/urdf/pexod_visuals_collisions.xacro (robot description, xacro)
@@ -3,17 +3,17 @@
   <!-- MATERIALS -->
   <material name="Blue">
-    <color rgba="0 0 1 1"/>
+    <color rgba="0.8 0.8 0.8 1.0"/>
     </material>
     <material name="Red">
-      <color rgba="1 0 0 1"/>
+      <color rgba="0.8 0.8 0.8 1.0"/>
     </material>
     <material name="Green">
-        <color rgba="0 1 0 1"/>
+        <color rgba="0.8 0.8 0.8 1.0"/>
   </material>
   <material name="Yellow">
-    <color rgba="1 1 0 1"/>
+    <color rgba="0.8 0.8 0.8 1.0"/>
     </material>
     <material name="LightGrey">
-      <color rgba="0.6 0.6 0.6 1.0"/>
+      <color rgba="0.8 0.8 0.8 1.0"/>
   </material>
     <!-- END OF MATERIALS -->
@@ -64,19 +64,37 @@
     </collision>
   </xacro:macro>
-  <xacro:macro name="visuals_collisions_leg_3" params="revert">
-    <visual>
-      <origin xyz="${leg3_width/2} ${revert*leg3_length/2} 0" rpy="${PI_2} 0 0"/>
-            <geometry>
-              <cylinder radius="${leg3_width}" length="${leg3_length}"/>
-            </geometry>
-      <material name="Red"/>
-    </visual>
-    <visual>
-      <origin xyz="${leg3_width/2} ${revert*leg3_length-revert*leg3_width/2} 0" rpy="${PI_2} 0 0"/>
-            <geometry>
-                <sphere radius="${leg3_width}"/>
-            </geometry>
-      <material name="Red"/>
-    </visual>
+  <xacro:macro name="visuals_collisions_leg_3" params="revert index">
+    <!-- <xacro:if value="${index == 5 or index == 4 or index == 3 or index == 2 or index == 0}"> -->
+      <visual>
+        <origin xyz="${leg3_width/2} ${revert*leg3_length/2} 0" rpy="${PI_2} 0 0"/>
+              <geometry>
+                <cylinder radius="${leg3_width}" length="${leg3_length}"/>
+              </geometry>
+        <material name="Red"/>
+      </visual>
+      <visual>
+        <origin xyz="${leg3_width/2} ${revert*leg3_length-revert*leg3_width/2} 0" rpy="${PI_2} 0 0"/>
+              <geometry>
+                  <sphere radius="${leg3_width}"/>
+              </geometry>
+        <material name="Red"/>
+      </visual>
+    <!-- </xacro:if>
+    <xacro:if value="${index == 1}">
+      <visual>
+        <origin xyz="${leg3_width/4} ${revert*leg3_length/4} 0" rpy="${PI_2} 0 0"/>
+              <geometry>
+                <cylinder radius="${leg3_width}" length="${leg3_length/2.0}"/>
+              </geometry>
+        <material name="Red"/>
+      </visual>
+      <visual>
+        <origin xyz="${leg3_width/4} ${revert*leg3_length/2.0-revert*leg3_width/4} 0" rpy="${PI_2} 0 0"/>
+              <geometry>
+                  <sphere radius="${leg3_width}"/>
+              </geometry>
+        <material name="Red"/>
+      </visual>
+    </xacro:if> -->
     <collision>
       <origin xyz="${leg3_width/2} ${revert*leg3_length/2} 0" rpy="${PI_2} 0 0"/>

Commit message: change length3

File: hexapod_description/urdf/modules/leg.xacro (robot description, xacro)
@@ -2,5 +2,5 @@
 <robot xmlns:xacro="http://www.ros.org/wiki/xacro">
   <!-- XACRO MACRO FOR LEGS LINKS/JOINTS -->
-    <xacro:macro name="leg" params="index xPos yPos sign">
+    <xacro:macro name="leg" params="index xPos yPos sign end_leg_lenght">
         <joint name="body_leg_${index}" type="revolute">
             <parent link="base_link"/>
@@ -71,11 +71,11 @@
         </joint>
         <link name="leg_${index}_3">
-            <xacro:visuals_collisions_leg_3 revert="${sign}" index="${index}"/>
+            <xacro:visuals_collisions_leg_3 revert="${sign}" index="${index}" end_leg_lenght="${end_leg_lenght}"/>
             <inertial>
                 <!-- CENTER OF MASS -->
-                <origin rpy="${PI_2} 0 0" xyz="${leg3_width/2} ${sign*leg3_length/2} 0"/>
+                <origin rpy="${PI_2} 0 0" xyz="${leg3_width/2} ${sign*end_leg_lenght/2} 0"/>
                 <mass value="${leg3_mass}"/>
                 <!-- box inertia: 1/12*m(y^2+z^2), ... -->
-                <inertia ixx="${1/12*leg3_mass*(leg3_width*leg3_width+leg3_length*leg3_length)}" ixy="0" ixz="0" iyy="${1/12*leg3_mass*(leg3_width*leg3_width+leg3_length*leg3_length)}" iyz="0" izz="${1/12*leg3_mass*(2*leg3_width*leg3_width)}"/>
+                <inertia ixx="${1/12*leg3_mass*(leg3_width*leg3_width+end_leg_lenght*end_leg_lenght)}" ixy="0" ixz="0" iyy="${1/12*leg3_mass*(leg3_width*leg3_width+end_leg_lenght*end_leg_lenght)}" iyz="0" izz="${1/12*leg3_mass*(2*leg3_width*leg3_width)}"/>
             </inertial>
         </link>

File: hexapod_description/urdf/modules/legs.xacro (robot description, xacro)
@@ -8,10 +8,10 @@
     <xacro:leg index="4" xPos="${-leg1_width/2}" yPos="${body_width/2}" sign="1"/>
     <xacro:leg index="1" xPos="${-leg1_width/2}" yPos="${-body_width/2}" sign="-1"/> -->
-    <xacro:leg index="2" xPos="${body_length/2-leg1_width/2}" yPos="${body_length/4}" sign="1"/>
-    <xacro:leg index="3" xPos="${body_length/2-leg1_width/2}" yPos="${-body_length/4}" sign="-1"/>
-    <xacro:leg index="0" xPos="${-body_length/2-leg1_width/2}" yPos="${body_length/4}" sign="1"/>
-    <xacro:leg index="5" xPos="${-body_length/2-leg1_width/2}" yPos="${-body_length/4}" sign="-1"/>
-    <xacro:leg index="1" xPos="${-leg1_width/2}" yPos="${body_width/2}" sign="1"/>
-    <xacro:leg index="4" xPos="${-leg1_width/2}" yPos="${-body_width/2}" sign="-1"/>
+    <xacro:leg index="2" xPos="${body_length/2-leg1_width/2}" yPos="${body_length/4}" sign="1" end_leg_lenght="${end_leg_lenght_2}"/>
+    <xacro:leg index="3" xPos="${body_length/2-leg1_width/2}" yPos="${-body_length/4}" sign="-1" end_leg_lenght="${end_leg_lenght_3}"/>
+    <xacro:leg index="0" xPos="${-body_length/2-leg1_width/2}" yPos="${body_length/4}" sign="1" end_leg_lenght="${end_leg_lenght_0}"/>
+    <xacro:leg index="5" xPos="${-body_length/2-leg1_width/2}" yPos="${-body_length/4}" sign="-1" end_leg_lenght="${end_leg_lenght_5}"/>
+    <xacro:leg index="1" xPos="${-leg1_width/2}" yPos="${body_width/2}" sign="1" end_leg_lenght="${end_leg_lenght_1}"/>
+    <xacro:leg index="4" xPos="${-leg1_width/2}" yPos="${-body_width/2}" sign="-1" end_leg_lenght="${end_leg_lenght_4}"/>
   <!-- END OF LEG LINKS/JOINTS -->
 </robot>

File: hexapod_description/urdf/modules/pexod.xacro (robot description, xacro)
@@ -27,10 +27,10 @@
   <xacro:property name="joint_vel" value="7.0"/>
   <xacro:property name="joint_dmp" value="0.0"/>
-  <xacro:property name="end_leg_lenght_0" value="0.140"/>
-  <xacro:property name="end_leg_lenght_1" value="0.140"/>
-  <xacro:property name="end_leg_lenght_2" value="0.140"/>
-  <xacro:property name="end_leg_lenght_3" value="0.140"/>
-  <xacro:property name="end_leg_lenght_4" value="0.140"/>
-  <xacro:property name="end_leg_lenght_5" value="0.140"/>
+  <xacro:property name="end_leg_lenght_0" value="0.195760642442"/>
+  <xacro:property name="end_leg_lenght_1" value="0.174571041985"/>
+  <xacro:property name="end_leg_lenght_2" value="0.173437213848"/>
+  <xacro:property name="end_leg_lenght_3" value="0.0445569955162"/>
+  <xacro:property name="end_leg_lenght_4" value="0.0405299416947"/>
+  <xacro:property name="end_leg_lenght_5" value="0.05605478672"/>
   <xacro:include filename="$(find hexapod_description)/urdf/pexod_visuals_collisions.xacro" />
   <!-- Load xacro modules/parts of the robot -->

File: hexapod_description/urdf/pexod.xacro (robot description, xacro)
@@ -2,4 +2,4 @@
 <robot name="pexod" xmlns:xacro="http://www.ros.org/wiki/xacro">
   <!-- <xacro:include filename="$(find pexod_description)/urdf/pexod_control.xacro" /> -->
-  <xacro:include filename="$(find hexapod_description)/urdf/modules/robot.xacro" />
+  <xacro:include filename="$(find hexapod_description)/urdf/modules/pexod.xacro" />
 </robot>

File: hexapod_description/urdf/pexod_visuals_collisions.xacro (robot description, xacro)
@@ -3,17 +3,17 @@
   <!-- MATERIALS -->
   <material name="Blue">
-    <color rgba="0.8 0.8 0.8 1.0"/>
-    </material>
-    <material name="Red">
-      <color rgba="0.8 0.8 0.8 1.0"/>
-    </material>
-    <material name="Green">
-        <color rgba="0.8 0.8 0.8 1.0"/>
+    <color rgba="0 0 1 1"/>
+  </material>
+  <material name="Red">
+    <color rgba="1 0 0 1"/>
+  </material>
+  <material name="Green">
+    <color rgba="0 1 0 1"/>
   </material>
   <material name="Yellow">
-    <color rgba="0.8 0.8 0.8 1.0"/>
-    </material>
-    <material name="LightGrey">
-      <color rgba="0.8 0.8 0.8 1.0"/>
+    <color rgba="1 1 0 1"/>
+  </material>
+  <material name="LightGrey">
+    <color rgba="0.6 0.6 0.6 1.0"/>
   </material>
     <!-- END OF MATERIALS -->
@@ -64,15 +64,14 @@
     </collision>
   </xacro:macro>
-  <xacro:macro name="visuals_collisions_leg_3" params="revert index">
-    <!-- <xacro:if value="${index == 5 or index == 4 or index == 3 or index == 2 or index == 0}"> -->
+  <xacro:macro name="visuals_collisions_leg_3" params="revert index end_leg_lenght">
       <visual>
-        <origin xyz="${leg3_width/2} ${revert*leg3_length/2} 0" rpy="${PI_2} 0 0"/>
+        <origin xyz="${leg3_width/2} ${revert*end_leg_lenght/2} 0" rpy="${PI_2} 0 0"/>
               <geometry>
-                <cylinder radius="${leg3_width}" length="${leg3_length}"/>
+                <cylinder radius="${leg3_width}" length="${end_leg_lenght}"/>
               </geometry>
         <material name="Red"/>
       </visual>
       <visual>
-        <origin xyz="${leg3_width/2} ${revert*leg3_length-revert*leg3_width/2} 0" rpy="${PI_2} 0 0"/>
+        <origin xyz="${leg3_width/2} ${revert*end_leg_lenght-revert*leg3_width/2} 0" rpy="${PI_2} 0 0"/>
               <geometry>
                   <sphere radius="${leg3_width}"/>
@@ -80,29 +79,12 @@
         <material name="Red"/>
       </visual>
-    <!-- </xacro:if>
-    <xacro:if value="${index == 1}">
-      <visual>
-        <origin xyz="${leg3_width/4} ${revert*leg3_length/4} 0" rpy="${PI_2} 0 0"/>
-              <geometry>
-                <cylinder radius="${leg3_width}" length="${leg3_length/2.0}"/>
-              </geometry>
-        <material name="Red"/>
-      </visual>
-      <visual>
-        <origin xyz="${leg3_width/4} ${revert*leg3_length/2.0-revert*leg3_width/4} 0" rpy="${PI_2} 0 0"/>
-              <geometry>
-                  <sphere radius="${leg3_width}"/>
-              </geometry>
-        <material name="Red"/>
-      </visual>
-    </xacro:if> -->
     <collision>
-      <origin xyz="${leg3_width/2} ${revert*leg3_length/2} 0" rpy="${PI_2} 0 0"/>
+      <origin xyz="${leg3_width/2} ${revert*end_leg_lenght/2} 0" rpy="${PI_2} 0 0"/>
             <geometry>
-                <box size="${leg3_width} ${leg3_width} ${leg3_length}"/>
+                <box size="${leg3_width} ${leg3_width} ${end_leg_lenght}"/>
             </geometry>
     </collision>
     <collision>
-      <origin xyz="${leg3_width/2} ${revert*leg3_length-revert*leg3_width/2} 0" rpy="${PI_2} 0 0"/>
+      <origin xyz="${leg3_width/2} ${revert*end_leg_lenght-revert*leg3_width/2} 0" rpy="${PI_2} 0 0"/>
             <geometry>
                 <sphere radius="${leg3_width}"/>

File: hexapod_description/urdf/results/pexod_4.urdf (robot description, URDF)
Before this commit: robot pexod, 20 links, 19 joints
Links:
- removed link body
- link base_link: mass None -> 1.031; geometry collision box size=0.24 0.2 0.04; visual box size=0.24 0.2 0.04
- link leg_0_3: geometry collision box size=0.025 0.025 0.195760642442; collision sphere radius=0.025
- link leg_1_3: geometry collision box size=0.025 0.025 0.174571041985; collision sphere radius=0.025
- link leg_2_3: geometry collision box size=0.025 0.025 0.173437213848; collision sphere radius=0.025
- link leg_3_3: geometry collision box size=0.025 0.025 0.0445569955162; collision sphere radius=0.025
- link leg_4_3: geometry collision box size=0.025 0.025 0.0405299416947; collision sphere radius=0.025
- link leg_5_3: geometry collision box size=0.025 0.025 0.05605478672; collision sphere radius=0.025
Joints:
- removed joint dummy
- joint body_leg_0: parent body -> base_link
- joint body_leg_1: parent body -> base_link
- joint body_leg_2: parent body -> base_link
- joint body_leg_3: parent body -> base_link
- joint body_leg_4: parent body -> base_link
- joint body_leg_5: parent body -> base_link
- joint leg_0_1_2: limit lower=-1.57079632679 upper=1.57079632679 effort=30.0 velocity=7.0 -> lower=-0.78539816339 upper=0.78539816339 effort=30.0 velocity=7.0
- joint leg_0_2_3: limit lower=-1.57079632679 upper=1.57079632679 effort=30.0 velocity=7.0 -> lower=-0.78539816339 upper=0.78539816339 effort=30.0 velocity=7.0
- joint leg_1_1_2: limit lower=-1.57079632679 upper=1.57079632679 effort=30.0 velocity=7.0 -> lower=-0.78539816339 upper=0.78539816339 effort=30.0 velocity=7.0
- joint leg_1_2_3: limit lower=-1.57079632679 upper=1.57079632679 effort=30.0 velocity=7.0 -> lower=-0.78539816339 upper=0.78539816339 effort=30.0 velocity=7.0
- joint leg_2_1_2: limit lower=-1.57079632679 upper=1.57079632679 effort=30.0 velocity=7.0 -> lower=-0.78539816339 upper=0.78539816339 effort=30.0 velocity=7.0
- joint leg_2_2_3: limit lower=-1.57079632679 upper=1.57079632679 effort=30.0 velocity=7.0 -> lower=-0.78539816339 upper=0.78539816339 effort=30.0 velocity=7.0
- joint leg_3_1_2: limit lower=-1.57079632679 upper=1.57079632679 effort=30.0 velocity=7.0 -> lower=-0.78539816339 upper=0.78539816339 effort=30.0 velocity=7.0
- joint leg_3_2_3: limit lower=-1.57079632679 upper=1.57079632679 effort=30.0 velocity=7.0 -> lower=-0.78539816339 upper=0.78539816339 effort=30.0 velocity=7.0
- joint leg_4_1_2: limit lower=-1.57079632679 upper=1.57079632679 effort=30.0 velocity=7.0 -> lower=-0.78539816339 upper=0.78539816339 effort=30.0 velocity=7.0
- joint leg_4_2_3: limit lower=-1.57079632679 upper=1.57079632679 effort=30.0 velocity=7.0 -> lower=-0.78539816339 upper=0.78539816339 effort=30.0 velocity=7.0
- joint leg_5_1_2: limit lower=-1.57079632679 upper=1.57079632679 effort=30.0 velocity=7.0 -> lower=-0.78539816339 upper=0.78539816339 effort=30.0 velocity=7.0
- joint leg_5_2_3: limit lower=-1.57079632679 upper=1.57079632679 effort=30.0 velocity=7.0 -> lower=-0.78539816339 upper=0.78539816339 effort=30.0 velocity=7.0
