Commit message: gene ok

File: hexapod_description/urdf/modules/leg.xacro (robot description, xacro)
@@ -2,5 +2,5 @@
 <robot xmlns:xacro="http://www.ros.org/wiki/xacro">
   <!-- XACRO MACRO FOR LEGS LINKS/JOINTS -->
-    <xacro:macro name="leg" params="index xPos yPos sign end_leg_lenght">
+    <xacro:macro name="leg" params="index xPos yPos sign end_leg_lenght mid_leg_lenght">
         <joint name="body_leg_${index}" type="revolute">
             <parent link="base_link"/>
@@ -48,11 +48,11 @@
         </joint>
         <link name="leg_${index}_2">
-            <xacro:visuals_collisions_leg_2 revert="${sign}"/>
+            <xacro:visuals_collisions_leg_2 revert="${sign}"  mid_leg_lenght="${mid_leg_lenght}"/>
             <inertial>
                 <!-- CENTER OF MASS -->
-                <origin rpy="${PI_2} 0 0" xyz="${leg2_width/2} ${sign*leg2_length/2} 0"/>
+                <origin rpy="${PI_2} 0 0" xyz="${leg2_width/2} ${sign*mid_leg_lenght/2} 0"/>
                 <mass value="${leg2_mass}"/>
                 <!-- box inertia: 1/12*m(y^2+z^2), ... -->
-                <inertia ixx="${1/12*leg2_mass*(leg2_width*leg2_width+leg2_length*leg2_length)}" ixy="0" ixz="0" iyy="${1/12*leg2_mass*(leg2_width*leg2_width+leg2_length*leg2_length)}" iyz="0" izz="${1/12*leg2_mass*(2*leg2_width*leg2_width)}"/>
+                <inertia ixx="${1/12*leg2_mass*(leg2_width*leg2_width+mid_leg_lenght*mid_leg_lenght)}" ixy="0" ixz="0" iyy="${1/12*leg2_mass*(leg2_width*leg2_width+mid_leg_lenght*mid_leg_lenght)}" iyz="0" izz="${1/12*leg2_mass*(2*leg2_width*leg2_width)}"/>
             </inertial>
         </link>
@@ -61,5 +61,5 @@
             <child link="leg_${index}_3"/>
             <limit effort="${joint_eff}" lower="${-joint_lim2}" upper="${joint_lim2}" velocity="${joint_vel}"/>
-            <origin rpy="${-sign*PI_2} 0 0" xyz="0 ${sign*leg2_length} 0"/>
+            <origin rpy="${-sign*PI_2} 0 0" xyz="0 ${sign*mid_leg_lenght} 0"/>
             <xacro:if value="${index == 5 or index == 4 or index == 3}">
                 <axis xyz="1 0 0"/>

File: hexapod_description/urdf/modules/legs.xacro (robot description, xacro)
@@ -8,10 +8,10 @@
     <xacro:leg index="4" xPos="${-leg1_width/2}" yPos="${body_width/2}" sign="1"/>
     <xacro:leg index="1" xPos="${-leg1_width/2}" yPos="${-body_width/2}" sign="-1"/> -->
-    <xacro:leg index="2" xPos="${body_length/2-leg1_width/2}" yPos="${body_length/4}" sign="1" end_leg_lenght="${end_leg_lenght_2}"/>
-    <xacro:leg index="3" xPos="${body_length/2-leg1_width/2}" yPos="${-body_length/4}" sign="-1" end_leg_lenght="${end_leg_lenght_3}"/>
-    <xacro:leg index="0" xPos="${-body_length/2-leg1_width/2}" yPos="${body_length/4}" sign="1" end_leg_lenght="${end_leg_lenght_0}"/>
-    <xacro:leg index="5" xPos="${-body_length/2-leg1_width/2}" yPos="${-body_length/4}" sign="-1" end_leg_lenght="${end_leg_lenght_5}"/>
-    <xacro:leg index="1" xPos="${-leg1_width/2}" yPos="${body_width/2}" sign="1" end_leg_lenght="${end_leg_lenght_1}"/>
-    <xacro:leg index="4" xPos="${-leg1_width/2}" yPos="${-body_width/2}" sign="-1" end_leg_lenght="${end_leg_lenght_4}"/>
+    <xacro:leg index="2" xPos="${body_length/2-leg1_width/2}" yPos="${body_length/4}" sign="1" end_leg_lenght="${end_leg_lenght_2}" mid_leg_lenght="${mid_leg_lenght_2}"/>
+    <xacro:leg index="3" xPos="${body_length/2-leg1_width/2}" yPos="${-body_length/4}" sign="-1" end_leg_lenght="${end_leg_lenght_3}" mid_leg_lenght="${mid_leg_lenght_3}"/>
+    <xacro:leg index="0" xPos="${-body_length/2-leg1_width/2}" yPos="${body_length/4}" sign="1" end_leg_lenght="${end_leg_lenght_0}" mid_leg_lenght="${mid_leg_lenght_0}"/>
+    <xacro:leg index="5" xPos="${-body_length/2-leg1_width/2}" yPos="${-body_length/4}" sign="-1" end_leg_lenght="${end_leg_lenght_5}" mid_leg_lenght="${mid_leg_lenght_5}"/>
+    <xacro:leg index="1" xPos="${-leg1_width/2}" yPos="${body_width/2}" sign="1" end_leg_lenght="${end_leg_lenght_1}" mid_leg_lenght="${mid_leg_lenght_1}"/>
+    <xacro:leg index="4" xPos="${-leg1_width/2}" yPos="${-body_width/2}" sign="-1" end_leg_lenght="${end_leg_lenght_4}" mid_leg_lenght="${mid_leg_lenght_4}"/>
   <!-- END OF LEG LINKS/JOINTS -->
 </robot>

File: hexapod_description/urdf/modules/pexod.xacro (robot description, xacro)
@@ -15,5 +15,5 @@
   <xacro:property name="leg1_mass" value="0.02"/>
   <xacro:property name="leg2_width" value="0.02"/>
-  <xacro:property name="leg2_length" value="0.085"/>
+  <!-- <xacro:property name="leg2_length" value="0.085"/> -->
   <xacro:property name="leg2_dist" value="0.2"/>
   <xacro:property name="leg2_mass" value="0.184"/>
@@ -27,10 +27,16 @@
   <xacro:property name="joint_vel" value="7.0"/>
   <xacro:property name="joint_dmp" value="0.0"/>
-  <xacro:property name="end_leg_lenght_0" value="0.195760642442"/>
-  <xacro:property name="end_leg_lenght_1" value="0.174571041985"/>
-  <xacro:property name="end_leg_lenght_2" value="0.173437213848"/>
-  <xacro:property name="end_leg_lenght_3" value="0.0445569955162"/>
-  <xacro:property name="end_leg_lenght_4" value="0.0405299416947"/>
-  <xacro:property name="end_leg_lenght_5" value="0.05605478672"/>
+  <xacro:property name="end_leg_lenght_0" value="0.1710724238"/>
+  <xacro:property name="end_leg_lenght_1" value="0.112832676842"/>
+  <xacro:property name="end_leg_lenght_2" value="0.118580396678"/>
+  <xacro:property name="end_leg_lenght_3" value="0.17121455382"/>
+  <xacro:property name="end_leg_lenght_4" value="0.132714081127"/>
+  <xacro:property name="end_leg_lenght_5" value="0.133089883124"/>
+  <xacro:property name="mid_leg_lenght_0" value="0.0606450913199"/>
+  <xacro:property name="mid_leg_lenght_1" value="0.06653684716"/>
+  <xacro:property name="mid_leg_lenght_2" value="0.0988183427764"/>
+  <xacro:property name="mid_leg_lenght_3" value="0.0916923999471"/>
+  <xacro:property name="mid_leg_lenght_4" value="0.0713142195319"/>
+  <xacro:property name="mid_leg_lenght_5" value="0.121756106183"/>
   <xacro:include filename="$(find hexapod_description)/urdf/pexod_visuals_collisions.xacro" />
   <!-- Load xacro modules/parts of the robot -->

File: hexapod_description/urdf/modules/robot.xacro (robot description, xacro)
@@ -15,5 +15,5 @@
   <xacro:property name="leg1_mass" value="0.02"/>
   <xacro:property name="leg2_width" value="0.02"/>
-  <xacro:property name="leg2_length" value="0.085"/>
+  <!-- <xacro:property name="leg2_length" value="0.085"/> -->
   <xacro:property name="leg2_dist" value="0.2"/>
   <xacro:property name="leg2_mass" value="0.184"/>
@@ -33,4 +33,10 @@
   <xacro:property name="end_leg_lenght_4" value="0.140"/>
   <xacro:property name="end_leg_lenght_5" value="0.140"/>
+  <xacro:property name="mid_leg_lenght_0" value="0.085"/>
+  <xacro:property name="mid_leg_lenght_1" value="0.085"/>
+  <xacro:property name="mid_leg_lenght_2" value="0.085"/>
+  <xacro:property name="mid_leg_lenght_3" value="0.085"/>
+  <xacro:property name="mid_leg_lenght_4" value="0.085"/>
+  <xacro:property name="mid_leg_lenght_5" value="0.085"/>
   <xacro:include filename="$(find hexapod_description)/urdf/pexod_visuals_collisions.xacro" />
   <!-- Load xacro modules/parts of the robot -->

File: hexapod_description/urdf/pexod_visuals_collisions.xacro (robot description, xacro)
@@ -49,16 +49,16 @@
     </collision>
   </xacro:macro>
-  <xacro:macro name="visuals_collisions_leg_2" params="revert">
+  <xacro:macro name="visuals_collisions_leg_2" params="revert mid_leg_lenght">
     <visual>
-      <origin xyz="${leg2_width/2} ${revert*leg2_length/2} 0" rpy="${PI_2} 0 0"/>
+      <origin xyz="${leg2_width/2} ${revert*mid_leg_lenght/2} 0" rpy="${PI_2} 0 0"/>
             <geometry>
-                <cylinder radius="${leg2_width}" length="${leg2_length}"/>
+                <cylinder radius="${leg2_width}" length="${mid_leg_lenght}"/>
             </geometry>
       <material name="Blue"/>
     </visual>
     <collision>
-      <origin xyz="${leg2_width/2} ${revert*leg2_length/2} 0" rpy="${PI_2} 0 0"/>
+      <origin xyz="${leg2_width/2} ${revert*mid_leg_lenght/2} 0" rpy="${PI_2} 0 0"/>
             <geometry>
-                <box size="${leg2_width} ${leg2_width} ${leg2_length}"/>
+                <box size="${leg2_width} ${leg2_width} ${mid_leg_lenght}"/>
             </geometry>
     </collision>

File: hexapod_description/urdf/results/pexod_0.urdf (robot description, URDF)
Before this commit: robot pexod, 19 links, 18 joints
Links:
- link leg_0_2: geometry collision box size=0.02 0.02 0.0876341422579; visual cylinder length=0.0876341422579 radius=0.02
- link leg_0_3: geometry collision box size=0.025 0.025 0.112685978747; collision sphere radius=0.025
- link leg_1_2: geometry collision box size=0.02 0.02 0.0946651550629; visual cylinder length=0.0946651550629 radius=0.02
- link leg_1_3: geometry collision box size=0.025 0.025 0.138099539471; collision sphere radius=0.025
- link leg_2_2: geometry collision box size=0.02 0.02 0.0975331078057; visual cylinder length=0.0975331078057 radius=0.02
- link leg_2_3: geometry collision box size=0.025 0.025 0.170662202522; collision sphere radius=0.025
- link leg_3_2: geometry collision box size=0.02 0.02 0.0539993327185; visual cylinder length=0.0539993327185 radius=0.02
- link leg_3_3: geometry collision box size=0.025 0.025 0.138487728849; collision sphere radius=0.025
- link leg_4_2: geometry collision box size=0.02 0.02 0.0568419481453; visual cylinder length=0.0568419481453 radius=0.02
- link leg_4_3: geometry collision box size=0.025 0.025 0.114810882451; collision sphere radius=0.025
- link leg_5_2: geometry collision box size=0.02 0.02 0.0482547367591; visual cylinder length=0.0482547367591 radius=0.02
- link leg_5_3: geometry collision box size=0.025 0.025 0.129473407241; collision sphere radius=0.025
Joints:
- joint leg_0_2_3: origin xyz=0 0.085 0 rpy=-1.57079632679 0 0 -> xyz=0 0.0876341422579 0 rpy=-1.57079632679 0 0
- joint leg_1_2_3: origin xyz=0 0.085 0 rpy=-1.57079632679 0 0 -> xyz=0 0.0946651550629 0 rpy=-1.57079632679 0 0
- joint leg_2_2_3: origin xyz=0 0.085 0 rpy=-1.57079632679 0 0 -> xyz=0 0.0975331078057 0 rpy=-1.57079632679 0 0
- joint leg_3_2_3: origin xyz=0 -0.085 0 rpy=1.57079632679 0 0 -> xyz=0 -0.0539993327185 0 rpy=1.57079632679 0 0
- joint leg_4_2_3: origin xyz=0 -0.085 0 rpy=1.57079632679 0 0 -> xyz=0 -0.0568419481453 0 rpy=1.57079632679 0 0
- joint leg_5_2_3: origin xyz=0 -0.085 0 rpy=1.57079632679 0 0 -> xyz=0 -0.0482547367591 0 rpy=1.57079632679 0 0

File: hexapod_description/urdf/results/pexod_1.urdf (robot description, URDF)
Before this commit: robot pexod, 19 links, 18 joints
Links:
- link leg_0_2: geometry collision box size=0.02 0.02 0.0555147427451; visual cylinder length=0.0555147427451 radius=0.02
- link leg_0_3: geometry collision box size=0.025 0.025 0.100065271625; collision sphere radius=0.025
- link leg_1_2: geometry collision box size=0.02 0.02 0.117559324683; visual cylinder length=0.117559324683 radius=0.02
- link leg_1_3: geometry collision box size=0.025 0.025 0.13757299749; collision sphere radius=0.025
- link leg_2_2: geometry collision box size=0.02 0.02 0.0739422578817; visual cylinder length=0.0739422578817 radius=0.02
- link leg_2_3: geometry collision box size=0.025 0.025 0.132699566973; collision sphere radius=0.025
- link leg_3_2: geometry collision box size=0.02 0.02 0.069868285568; visual cylinder length=0.069868285568 radius=0.02
- link leg_3_3: geometry collision box size=0.025 0.025 0.162992334522; collision sphere radius=0.025
- link leg_4_2: geometry collision box size=0.02 0.02 0.0471756559122; visual cylinder length=0.0471756559122 radius=0.02
- link leg_4_3: geometry collision box size=0.025 0.025 0.17150028976; collision sphere radius=0.025
- link leg_5_2: geometry collision box size=0.02 0.02 0.0770272278217; visual cylinder length=0.0770272278217 radius=0.02
- link leg_5_3: geometry collision box size=0.025 0.025 0.174196485609; collision sphere radius=0.025
Joints:
- joint leg_0_2_3: origin xyz=0 0.085 0 rpy=-1.57079632679 0 0 -> xyz=0 0.0555147427451 0 rpy=-1.57079632679 0 0
- joint leg_1_2_3: origin xyz=0 0.085 0 rpy=-1.57079632679 0 0 -> xyz=0 0.117559324683 0 rpy=-1.57079632679 0 0
- joint leg_2_2_3: origin xyz=0 0.085 0 rpy=-1.57079632679 0 0 -> xyz=0 0.0739422578817 0 rpy=-1.57079632679 0 0
- joint leg_3_2_3: origin xyz=0 -0.085 0 rpy=1.57079632679 0 0 -> xyz=0 -0.069868285568 0 rpy=1.57079632679 0 0
- joint leg_4_2_3: origin xyz=0 -0.085 0 rpy=1.57079632679 0 0 -> xyz=0 -0.0471756559122 0 rpy=1.57079632679 0 0
- joint leg_5_2_3: origin xyz=0 -0.085 0 rpy=1.57079632679 0 0 -> xyz=0 -0.0770272278217 0 rpy=1.57079632679 0 0

File: hexapod_description/urdf/results/pexod_2.urdf (robot description, URDF)
Before this commit: robot pexod, 19 links, 18 joints
Links:
- link leg_0_2: geometry collision box size=0.02 0.02 0.0795076727308; visual cylinder length=0.0795076727308 radius=0.02
- link leg_0_3: geometry collision box size=0.025 0.025 0.15999315651; collision sphere radius=0.025
- link leg_1_2: geometry collision box size=0.02 0.02 0.0868091333757; visual cylinder length=0.0868091333757 radius=0.02
- link leg_1_3: geometry collision box size=0.025 0.025 0.156490851333; collision sphere radius=0.025
- link leg_2_2: geometry collision box size=0.02 0.02 0.0780631302782; visual cylinder length=0.0780631302782 radius=0.02
- link leg_2_3: geometry collision box size=0.025 0.025 0.106251187281; collision sphere radius=0.025
- link leg_3_2: geometry collision box size=0.02 0.02 0.0455315950465; visual cylinder length=0.0455315950465 radius=0.02
- link leg_3_3: geometry collision box size=0.025 0.025 0.168896267114; collision sphere radius=0.025
- link leg_4_2: geometry collision box size=0.02 0.02 0.12119386186; visual cylinder length=0.12119386186 radius=0.02
- link leg_4_3: geometry collision box size=0.025 0.025 0.12940123232; collision sphere radius=0.025
- link leg_5_2: geometry collision box size=0.02 0.02 0.104359810496; visual cylinder length=0.104359810496 radius=0.02
- link leg_5_3: geometry collision box size=0.025 0.025 0.162315119796; collision sphere radius=0.025
Joints:
- joint leg_0_2_3: origin xyz=0 0.085 0 rpy=-1.57079632679 0 0 -> xyz=0 0.0795076727308 0 rpy=-1.57079632679 0 0
- joint leg_1_2_3: origin xyz=0 0.085 0 rpy=-1.57079632679 0 0 -> xyz=0 0.0868091333757 0 rpy=-1.57079632679 0 0
- joint leg_2_2_3: origin xyz=0 0.085 0 rpy=-1.57079632679 0 0 -> xyz=0 0.0780631302782 0 rpy=-1.57079632679 0 0
- joint leg_3_2_3: origin xyz=0 -0.085 0 rpy=1.57079632679 0 0 -> xyz=0 -0.0455315950465 0 rpy=1.57079632679 0 0
- joint leg_4_2_3: origin xyz=0 -0.085 0 rpy=1.57079632679 0 0 -> xyz=0 -0.12119386186 0 rpy=1.57079632679 0 0
- joint leg_5_2_3: origin xyz=0 -0.085 0 rpy=1.57079632679 0 0 -> xyz=0 -0.104359810496 0 rpy=1.57079632679 0 0

File: hexapod_description/urdf/results/pexod_3.urdf (robot description, URDF)
Before this commit: robot pexod, 19 links, 18 joints
Links:
- link leg_0_2: geometry collision box size=0.02 0.02 0.0671556191779; visual cylinder length=0.0671556191779 radius=0.02
- link leg_0_3: geometry collision box size=0.025 0.025 0.119951042505; collision sphere radius=0.025
- link leg_1_2: geometry collision box size=0.02 0.02 0.100126030573; visual cylinder length=0.100126030573 radius=0.02
- link leg_1_3: geometry collision box size=0.025 0.025 0.153759559156; collision sphere radius=0.025
- link leg_2_2: geometry collision box size=0.02 0.02 0.046004135085; visual cylinder length=0.046004135085 radius=0.02
- link leg_2_3: geometry collision box size=0.025 0.025 0.153618303182; collision sphere radius=0.025
- link leg_3_2: geometry collision box size=0.02 0.02 0.0913690701209; visual cylinder length=0.0913690701209 radius=0.02
- link leg_3_3: geometry collision box size=0.025 0.025 0.107128470221; collision sphere radius=0.025
- link leg_4_2: geometry collision box size=0.02 0.02 0.096734935374; visual cylinder length=0.096734935374 radius=0.02
- link leg_4_3: geometry collision box size=0.025 0.025 0.126073946257; collision sphere radius=0.025
- link leg_5_2: geometry collision box size=0.02 0.02 0.106647218271; visual cylinder length=0.106647218271 radius=0.02
- link leg_5_3: geometry collision box size=0.025 0.025 0.141171576038; collision sphere radius=0.025
Joints:
- joint leg_0_2_3: origin xyz=0 0.085 0 rpy=-1.57079632679 0 0 -> xyz=0 0.0671556191779 0 rpy=-1.57079632679 0 0
- joint leg_1_2_3: origin xyz=0 0.085 0 rpy=-1.57079632679 0 0 -> xyz=0 0.100126030573 0 rpy=-1.57079632679 0 0
- joint leg_2_2_3: origin xyz=0 0.085 0 rpy=-1.57079632679 0 0 -> xyz=0 0.046004135085 0 rpy=-1.57079632679 0 0
- joint leg_3_2_3: origin xyz=0 -0.085 0 rpy=1.57079632679 0 0 -> xyz=0 -0.0913690701209 0 rpy=1.57079632679 0 0
- joint leg_4_2_3: origin xyz=0 -0.085 0 rpy=1.57079632679 0 0 -> xyz=0 -0.096734935374 0 rpy=1.57079632679 0 0
- joint leg_5_2_3: origin xyz=0 -0.085 0 rpy=1.57079632679 0 0 -> xyz=0 -0.106647218271 0 rpy=1.57079632679 0 0

File: hexapod_description/urdf/results/pexod_4.urdf (robot description, URDF)
Before this commit: robot pexod, 19 links, 18 joints
Links:
- link leg_0_2: geometry collision box size=0.02 0.02 0.0800961129833; visual cylinder length=0.0800961129833 radius=0.02
- link leg_0_3: geometry collision box size=0.025 0.025 0.106537640913; collision sphere radius=0.025
- link leg_1_2: geometry collision box size=0.02 0.02 0.0631748524181; visual cylinder length=0.0631748524181 radius=0.02
- link leg_1_3: geometry collision box size=0.025 0.025 0.125443799126; collision sphere radius=0.025
- link leg_2_2: geometry collision box size=0.02 0.02 0.122268029567; visual cylinder length=0.122268029567 radius=0.02
- link leg_2_3: geometry collision box size=0.025 0.025 0.161282691369; collision sphere radius=0.025
- link leg_3_2: geometry collision box size=0.02 0.02 0.11419129676; visual cylinder length=0.11419129676 radius=0.02
- link leg_3_3: geometry collision box size=0.025 0.025 0.165129558306; collision sphere radius=0.025
- link leg_4_2: geometry collision box size=0.02 0.02 0.0627124292571; visual cylinder length=0.0627124292571 radius=0.02
- link leg_4_3: geometry collision box size=0.025 0.025 0.129887579702; collision sphere radius=0.025
- link leg_5_2: geometry collision box size=0.02 0.02 0.0926637902545; visual cylinder length=0.0926637902545 radius=0.02
- link leg_5_3: geometry collision box size=0.025 0.025 0.115360355214; collision sphere radius=0.025
Joints:
- joint leg_0_2_3: origin xyz=0 0.085 0 rpy=-1.57079632679 0 0 -> xyz=0 0.0800961129833 0 rpy=-1.57079632679 0 0
- joint leg_1_2_3: origin xyz=0 0.085 0 rpy=-1.57079632679 0 0 -> xyz=0 0.0631748524181 0 rpy=-1.57079632679 0 0
- joint leg_2_2_3: origin xyz=0 0.085 0 rpy=-1.57079632679 0 0 -> xyz=0 0.122268029567 0 rpy=-1.57079632679 0 0
- joint leg_3_2_3: origin xyz=0 -0.085 0 rpy=1.57079632679 0 0 -> xyz=0 -0.11419129676 0 rpy=1.57079632679 0 0
- joint leg_4_2_3: origin xyz=0 -0.085 0 rpy=1.57079632679 0 0 -> xyz=0 -0.0627124292571 0 rpy=1.57079632679 0 0
- joint leg_5_2_3: origin xyz=0 -0.085 0 rpy=1.57079632679 0 0 -> xyz=0 -0.0926637902545 0 rpy=1.57079632679 0 0
