Commit message: Boxes for collision - should change the inertia properties

File: hexapod_description/urdf/pexod_visuals_collisions.xacro (robot description, xacro)
@@ -45,5 +45,5 @@
 			<origin xyz="${leg1_width/2} ${revert*leg1_length/2} 0" rpy="${PI_2} 0 0"/>
             <geometry>
-                <cylinder radius="${leg1_width}" length="${leg1_length}"/>
+                <box size="${1.5*leg1_width} ${1.5*leg1_width} ${leg1_length}"/>
             </geometry>
 		</collision>
@@ -60,5 +60,5 @@
 			<origin xyz="${leg2_width/2} ${revert*leg2_length/2} 0" rpy="${PI_2} 0 0"/>
             <geometry>
-                <cylinder radius="${leg2_width}" length="${leg2_length}"/>
+                <box size="${1.5*leg2_width} ${1.5*leg2_width} ${leg2_length}"/>
             </geometry>
 		</collision>
@@ -68,5 +68,5 @@
 			<origin xyz="${leg3_width/2} ${revert*leg3_length/2} 0" rpy="${PI_2} 0 0"/>
             <geometry>
-                <cylinder radius="${leg3_width}" length="${leg3_length-leg3_width}"/>
+              <cylinder radius="${leg3_width}" length="${leg3_length}"/>
             </geometry>
 			<material name="Red"/>
@@ -82,5 +82,5 @@
 			<origin xyz="${leg3_width/2} ${revert*leg3_length/2} 0" rpy="${PI_2} 0 0"/>
             <geometry>
-                <cylinder radius="${leg3_width}" length="${leg3_length-leg3_width}"/>
+                <box size="${1.5*leg3_width} ${1.5*leg3_width} ${leg3_length}"/>
             </geometry>
 		</collision>

Commit message: fix x shift in visual and collision geometries

File: hexapod_description/urdf/pexod_visuals_collisions.xacro (robot description, xacro)
@@ -27,4 +27,11 @@
       <material name="Blue"/>
     </visual>
+    <visual>
+      <origin xyz="0 0 0" rpy="0 0 0"/>
+            <geometry>
+                <box size="${leg1_width*2.5} ${body_width_extra} ${body_height}"/>
+            </geometry>
+      <material name="Blue"/>
+    </visual>
     <collision>
       <origin xyz="0 0 0" rpy="0 0 0"/>
@@ -36,5 +43,5 @@
   <xacro:macro name="visuals_collisions_leg_1" params="revert">
     <visual>
-      <origin xyz="${leg1_width/2} ${revert*leg1_length/2} 0" rpy="${PI_2} 0 0"/>
+      <origin xyz="0 ${revert*leg1_length/2} 0" rpy="${PI_2} 0 0"/>
             <geometry>
                 <cylinder radius="${leg1_width}" length="${leg1_length}"/>
@@ -43,5 +50,5 @@
     </visual>
     <collision>
-      <origin xyz="${leg1_width/2} ${revert*leg1_length/2} 0" rpy="${PI_2} 0 0"/>
+      <origin xyz="0 ${revert*leg1_length/2} 0" rpy="${PI_2} 0 0"/>
             <geometry>
                 <box size="${leg1_width} ${leg1_width} ${leg1_length}"/>
@@ -51,5 +58,5 @@
   <xacro:macro name="visuals_collisions_leg_2" params="revert">
     <visual>
-      <origin xyz="${leg2_width/2} ${revert*leg2_length/2} 0" rpy="${PI_2} 0 0"/>
+      <origin xyz="0 ${revert*leg2_length/2} 0" rpy="${PI_2} 0 0"/>
             <geometry>
                 <cylinder radius="${leg2_width}" length="${leg2_length}"/>
@@ -58,5 +65,5 @@
     </visual>
     <collision>
-      <origin xyz="${leg2_width/2} ${revert*leg2_length/2} 0" rpy="${PI_2} 0 0"/>
+      <origin xyz="0 ${revert*leg2_length/2} 0" rpy="${PI_2} 0 0"/>
             <geometry>
                 <box size="${leg2_width} ${leg2_width} ${leg2_length}"/>
@@ -66,5 +73,5 @@
   <xacro:macro name="visuals_collisions_leg_3" params="revert">
     <visual>
-      <origin xyz="${leg3_width/2} ${revert*leg3_length/2} 0" rpy="${PI_2} 0 0"/>
+      <origin xyz="0 ${revert*leg3_length/2} 0" rpy="${PI_2} 0 0"/>
             <geometry>
               <cylinder radius="${leg3_width}" length="${leg3_length}"/>
@@ -73,5 +80,5 @@
     </visual>
     <visual>
-      <origin xyz="${leg3_width/2} ${revert*leg3_length-revert*leg3_width/2} 0" rpy="${PI_2} 0 0"/>
+      <origin xyz="0 ${revert*leg3_length-revert*leg3_width/2} 0" rpy="${PI_2} 0 0"/>
             <geometry>
                 <sphere radius="${leg3_width}"/>
@@ -80,5 +87,5 @@
     </visual>
     <collision>
-      <origin xyz="${leg3_width/2} ${revert*leg3_length/2} 0" rpy="${PI_2} 0 0"/>
+      <origin xyz="0 ${revert*leg3_length/2} 0" rpy="${PI_2} 0 0"/>
             <geometry>
                 <box size="${leg3_width} ${leg3_width} ${leg3_length}"/>
@@ -86,5 +93,5 @@
     </collision>
     <collision>
-      <origin xyz="${leg3_width/2} ${revert*leg3_length-revert*leg3_width/2} 0" rpy="${PI_2} 0 0"/>
+      <origin xyz="0 ${revert*leg3_length-revert*leg3_width/2} 0" rpy="${PI_2} 0 0"/>
             <geometry>
                 <sphere radius="${leg3_width}"/>

Commit message: change colour of pexod's body

File: hexapod_description/urdf/pexod_visuals_collisions.xacro (robot description, xacro)
@@ -15,5 +15,5 @@
     </material>
     <material name="LightGrey">
-      <color rgba="0.6 0.6 0.6 1.0"/>
+      <color rgba="0.5 0.5 0.85 1.0"/>
   </material>
     <!-- END OF MATERIALS -->
@@ -25,5 +25,5 @@
                 <box size="${body_length} ${body_width} ${body_height}"/>
             </geometry>
-      <material name="Blue"/>
+      <material name="LightGrey"/>
     </visual>
     <visual>
@@ -32,5 +32,5 @@
                 <box size="${leg1_width*2.5} ${body_width_extra} ${body_height}"/>
             </geometry>
-      <material name="Blue"/>
+      <material name="LightGrey"/>
     </visual>
     <collision>
