Commit message: update collision geometries to match visuals

File: hexapod_description/urdf/marta_visuals_collisions.xacro (robot description, xacro)
@@ -38,4 +38,10 @@
             <geometry>
                 <box size="${body_length} ${body_width} ${body_height}"/>
+            </geometry>
+    </collision>
+    <collision>
+      <origin xyz="0 0 0" rpy="0 0 0"/>
+            <geometry>
+                <box size="${leg1_width*2.5} ${body_width_extra} ${body_height}"/>
             </geometry>
     </collision>
@@ -103,11 +109,20 @@
     </visual>
     <collision>
-      <origin xyz="0 ${revert*leg3_length/2} 0" rpy="${PI_2} 0 0"/>
+      <origin xyz="0 0 ${leg3_dist/2}" rpy="0 0 0"/>
             <geometry>
-                <box size="${leg3_width} ${leg3_width} ${leg3_length}"/>
+              <box size="${leg3_width} ${leg3_width} ${leg3_dist}"/>
             </geometry>
+      <material name="Red"/>
     </collision>
     <collision>
-      <origin xyz="0 ${revert*leg3_length-revert*leg3_width/2} 0"
+      <origin xyz="0 ${revert*leg3_length/2} ${leg3_dist}"
+        rpy="${PI_2} 0 0"/>
+            <geometry>
+              <box size="${leg3_width} ${leg3_width} ${leg3_length}"/>
+            </geometry>
+      <material name="Red"/>
+    </collision>
+    <collision>
+      <origin xyz="0 ${revert*leg3_length-revert*leg3_width/2} ${leg3_dist}"
         rpy="${PI_2} 0 0"/>
             <geometry>

File: hexapod_description/urdf/pexod_visuals_collisions.xacro (robot description, xacro)
@@ -38,4 +38,10 @@
             <geometry>
                 <box size="${body_length} ${body_width} ${body_height}"/>
+            </geometry>
+    </collision>
+    <collision>
+      <origin xyz="0 0 0" rpy="0 0 0"/>
+            <geometry>
+                <box size="${leg1_width*2.5} ${body_width_extra} ${body_height}"/>
             </geometry>
     </collision>

Commit message: adjust diameters of limbs

File: hexapod_description/urdf/marta_visuals_collisions.xacro (robot description, xacro)
@@ -51,5 +51,5 @@
       <origin xyz="0 ${revert*leg1_length/2} 0" rpy="${PI_2} 0 0"/>
             <geometry>
-                <cylinder radius="${leg1_width}" length="${leg1_length}"/>
+                <cylinder radius="${leg1_width/2}" length="${leg1_length}"/>
             </geometry>
       <material name="Red"/>
@@ -66,5 +66,5 @@
       <origin xyz="0 ${revert*leg2_length/2} 0" rpy="${PI_2} 0 0"/>
             <geometry>
-                <cylinder radius="${leg2_width}" length="${leg2_length}"/>
+                <cylinder radius="${leg2_width/2}" length="${leg2_length}"/>
             </geometry>
       <material name="Blue"/>
@@ -81,5 +81,5 @@
       <origin xyz="0 0 ${leg3_dist/2}" rpy="0 0 0"/>
             <geometry>
-              <cylinder radius="${leg3_width}" length="${leg3_dist}"/>
+              <cylinder radius="${leg3_width/2}" length="${leg3_dist}"/>
             </geometry>
       <material name="Red"/>
@@ -88,5 +88,5 @@
       <origin xyz="0 0 ${leg3_dist}" rpy="0 0 0"/>
             <geometry>
-              <sphere radius="${leg3_width}"/>
+              <sphere radius="${leg3_width/2}"/>
             </geometry>
       <material name="Red"/>
@@ -96,13 +96,13 @@
         rpy="${PI_2} 0 0"/>
             <geometry>
-              <cylinder radius="${leg3_width}" length="${leg3_length}"/>
+              <cylinder radius="${leg3_width/2}" length="${leg3_length-leg3_tip_radius}"/>
             </geometry>
       <material name="Red"/>
     </visual>
     <visual>
-      <origin xyz="0 ${revert*leg3_length-revert*leg3_width/2} ${leg3_dist}"
+      <origin xyz="0 ${revert*leg3_length-revert*leg3_tip_radius} ${leg3_dist}"
         rpy="${PI_2} 0 0"/>
             <geometry>
-                <sphere radius="${leg3_width}"/>
+                <sphere radius="${leg3_tip_radius}"/>
             </geometry>
       <material name="Red"/>
@@ -111,5 +111,5 @@
       <origin xyz="0 0 ${leg3_dist/2}" rpy="0 0 0"/>
             <geometry>
-              <box size="${leg3_width} ${leg3_width} ${leg3_dist}"/>
+              <box size="${leg3_width} ${leg3_width} ${leg3_dist+leg3_width}"/>
             </geometry>
       <material name="Red"/>
@@ -119,13 +119,13 @@
         rpy="${PI_2} 0 0"/>
             <geometry>
-              <box size="${leg3_width} ${leg3_width} ${leg3_length}"/>
+              <box size="${leg3_width} ${leg3_width} ${leg3_length-leg3_tip_radius}"/>
             </geometry>
       <material name="Red"/>
     </collision>
     <collision>
-      <origin xyz="0 ${revert*leg3_length-revert*leg3_width/2} ${leg3_dist}"
+      <origin xyz="0 ${revert*leg3_length-revert*leg3_tip_radius} ${leg3_dist}"
         rpy="${PI_2} 0 0"/>
             <geometry>
-                <sphere radius="${leg3_width}"/>
+                <sphere radius="${leg3_tip_radius}"/>
             </geometry>
       <material name="Red"/>

File: hexapod_description/urdf/modules/marta.xacro (robot description, xacro)
@@ -11,15 +11,16 @@
   <xacro:property name="body_width_extra" value="0.190"/>
   <xacro:property name="body_height" value="0.04"/>
-  <xacro:property name="leg1_width" value="0.02"/>
+  <xacro:property name="leg1_width" value="0.05"/>
   <xacro:property name="leg1_length" value="0.06"/>
   <xacro:property name="leg1_dist" value="0.2"/>
   <xacro:property name="leg1_mass" value="0.02"/>
-  <xacro:property name="leg2_width" value="0.02"/>
+  <xacro:property name="leg2_width" value="0.05"/>
   <xacro:property name="leg2_length" value="0.0835"/>
   <xacro:property name="leg2_dist" value="0.2"/>
   <xacro:property name="leg2_mass" value="0.184"/>
-  <xacro:property name="leg3_width" value="0.02"/>
+  <xacro:property name="leg3_width" value="0.054"/>
   <xacro:property name="leg3_length" value="0.12"/>
   <xacro:property name="leg3_dist" value="0.038"/>
+  <xacro:property name="leg3_tip_radius" value="0.02"/>
   <xacro:property name="leg3_mass" value="0.04"/>
   <xacro:property name="joint_lim" value="${PI_2}"/>

Commit message: Add visual element to differentiate front and back of the robot

File: hexapod_description/urdf/marta_visuals_collisions.xacro (robot description, xacro)
@@ -12,7 +12,7 @@
   </material>
   <material name="Yellow">
-    <color rgba="1 1 0 1"/>
-    </material>
-    <material name="LightGrey">
+    <color rgba="0.8 0.9 0.3 1"/>
+  </material>
+  <material name="LightGrey">
       <color rgba="0.6 0.6 0.6 1.0"/>
   </material>
@@ -25,5 +25,5 @@
                 <box size="${body_length} ${body_width} ${body_height}"/>
             </geometry>
-      <material name="Blue"/>
+      <material name="Yellow"/>
     </visual>
     <visual>
@@ -46,4 +46,13 @@
             </geometry>
     </collision>
+  </xacro:macro>
+  <xacro:macro name="visuals_head" params="">
+    <visual>
+      <origin xyz="${body_length/2.} 0 ${body_height*0.7}" rpy="0 0 ${PI/4}"/>
+      <geometry>
+        <box size="${body_width/2.} ${body_width/2.} ${body_height*0.7}"/>
+      </geometry>
+      <material name="Yellow"/>
+    </visual>
   </xacro:macro>
   <xacro:macro name="visuals_collisions_leg_1" params="revert">

File: hexapod_description/urdf/modules/body.xacro (robot description, xacro)
@@ -4,4 +4,5 @@
     <link name="base_link">
         <xacro:visuals_collisions_body/>
+        <xacro:visuals_head/>
         <inertial>
             <!-- CENTER OF MASS -->

File: hexapod_description/urdf/pexod_visuals_collisions.xacro (robot description, xacro)
@@ -46,4 +46,13 @@
             </geometry>
     </collision>
+  </xacro:macro>
+  <xacro:macro name="visuals_head" params="">
+    <visual>
+      <origin xyz="${body_length/2.} 0 ${body_height*0.7}" rpy="0 0 ${PI/4}"/>
+      <geometry>
+        <box size="${body_width/2.} ${body_width/2.} ${body_height*0.7}"/>
+      </geometry>
+      <material name="Yellow"/>
+    </visual>
   </xacro:macro>
   <xacro:macro name="visuals_collisions_leg_1" params="revert">

Commit message: Actual 3D models for Hexaforce robot added

File: hexapod_description/urdf/marta_visuals_collisions.xacro (robot description, xacro)
@@ -21,16 +21,9 @@
     <xacro:macro name="visuals_collisions_body" params="">
     <visual>
-      <origin xyz="0 0 0" rpy="0 0 0"/>
-            <geometry>
-                <box size="${body_length} ${body_width} ${body_height}"/>
-            </geometry>
+      <origin xyz="0 0 0" rpy="${PI_2} 0 ${PI_2}"/>
+        <geometry>
+          <mesh filename="package://hexapod_description/stl/chassis.stl" scale="0.001 0.001 0.001"/>
+        </geometry>
       <material name="Yellow"/>
-    </visual>
-    <visual>
-      <origin xyz="0 0 0" rpy="0 0 0"/>
-            <geometry>
-                <box size="${leg1_width*2.5} ${body_width_extra} ${body_height}"/>
-            </geometry>
-      <material name="Blue"/>
     </visual>
     <collision>
@@ -49,89 +42,66 @@
   <xacro:macro name="visuals_head" params="">
     <visual>
-      <origin xyz="${body_length/2.} 0 ${body_height*0.7}" rpy="0 0 ${PI/4}"/>
+      <origin xyz="${body_length/2.} 0 0" rpy="0 0 ${PI/4}"/>
       <geometry>
-        <box size="${body_width/2.} ${body_width/2.} ${body_height*0.7}"/>
+        <box size="${body_width/3.} ${body_width/3.} ${body_height*0.6}"/>
       </geometry>
       <material name="Yellow"/>
     </visual>
   </xacro:macro>
-  <xacro:macro name="visuals_collisions_leg_1" params="revert">
+  <xacro:macro name="visuals_collisions_leg_1">
     <visual>
-      <origin xyz="0 ${revert*leg1_length/2} 0" rpy="${PI_2} 0 0"/>
-            <geometry>
-                <cylinder radius="${leg1_width/2}" length="${leg1_length}"/>
-            </geometry>
+      <origin xyz="0 0 0" rpy="0 ${PI_2} 0"/>
+        <geometry>
+          <mesh filename="package://hexapod_description/stl/first_link.stl" scale="0.001 0.001 0.001"/>
+        </geometry>
       <material name="Red"/>
     </visual>
     <collision>
-      <origin xyz="0 ${revert*leg1_length/2} 0" rpy="${PI_2} 0 0"/>
-            <geometry>
-                <box size="${leg1_width} ${leg1_width} ${leg1_length}"/>
-            </geometry>
+      <origin xyz="0 ${leg1_length/2} 0" rpy="${PI_2} 0 0"/>
+        <geometry>
+          <box size="${leg1_width} ${leg1_width} ${leg1_length}"/>
+        </geometry>
     </collision>
   </xacro:macro>
-  <xacro:macro name="visuals_collisions_leg_2" params="revert">
+  <xacro:macro name="visuals_collisions_leg_2">
     <visual>
-      <origin xyz="0 ${revert*leg2_length/2} 0" rpy="${PI_2} 0 0"/>
-            <geometry>
-                <cylinder radius="${leg2_width/2}" length="${leg2_length}"/>
-            </geometry>
+      <origin xyz="0 0 0" rpy="0 -${PI_2} 0"/>
+        <geometry>
+          <mesh filename="package://hexapod_description/stl/second_link.stl" scale="0.001 0.001 0.001"/>
+        </geometry>
       <material name="Blue"/>
     </visual>
     <collision>
-      <origin xyz="0 ${revert*leg2_length/2} 0" rpy="${PI_2} 0 0"/>
-            <geometry>
-                <box size="${leg2_width} ${leg2_width} ${leg2_length}"/>
-            </geometry>
+      <origin xyz="0 ${leg2_length/2} 0" rpy="${PI_2} 0 0"/>
+        <geometry>
+          <box size="${leg2_width} ${leg2_width} ${leg2_length}"/>
+        </geometry>
     </collision>
   </xacro:macro>
-  <xacro:macro name="visuals_collisions_leg_3" params="revert">
+  <xacro:macro name="visuals_collisions_leg_3">
     <visual>
-      <origin xyz="0 0 ${leg3_dist/2}" rpy="0 0 0"/>
-            <geometry>
-              <cylinder radius="${leg3_width/2}" length="${leg3_dist}"/>
-            </geometry>
-      <material name="Red"/>
-    </visual>
-    <visual>
-      <origin xyz="0 0 ${leg3_dist}" rpy="0 0 0"/>
-            <geometry>
-              <sphere radius="${leg3_width/2}"/>
-            </geometry>
-      <material name="Red"/>
-    </visual>
-    <visual>
-      <origin xyz="0 ${revert*leg3_length/2} ${leg3_dist}"
-        rpy="${PI_2} 0 0"/>
-            <geometry>
-              <cylinder radius="${leg3_width/2}" length="${leg3_length-leg3_tip_radius}"/>
-            </geometry>
-      <material name="Red"/>
-    </visual>
-    <visual>
-      <origin xyz="0 ${revert*leg3_length-revert*leg3_tip_radius} ${leg3_dist}"
-        rpy="${PI_2} 0 0"/>
-            <geometry>
-                <sphere radius="${leg3_tip_radius}"/>
-            </geometry>
-      <material name="Red"/>
+      <origin xyz="0 0 0" rpy="0 0 ${PI}"/>
+      <geometry>
+        <mesh filename="package://hexapod_description/stl/third_link.stl" scale="0.001 0.001 0.001"/>
+        <material name="Red"/>
+      </geometry>
     </visual>
     <collision>
-      <origin xyz="0 0 ${leg3_dist/2}" rpy="0 0 0"/>
-            <geometry>
-              <box size="${leg3_width} ${leg3_width} ${leg3_dist+leg3_width}"/>
-            </geometry>
+      <origin xyz="0 ${leg3_dist} 0" rpy="0 0 0"/>
+        <geometry>
+          <box size="${leg3_width} ${leg3_length} ${leg3_width}"/>
+        </geometry>
       <material name="Red"/>
     </collision>
     <collision>
-      <origin xyz="0 ${revert*leg3_length/2} ${leg3_dist}"
-        rpy="${PI_2} 0 0"/>
-            <geometry>
-              <box size="${leg3_width} ${leg3_width} ${leg3_length-leg3_tip_radius}"/>
-            </geometry>
+      <origin xyz="0 ${leg3_length-leg3_width/2} ${-(leg3_width+leg3_height-leg3_tip_radius)/2}"
+        rpy="0 0 0"/>
+        <geometry>
+          <box size="${leg3_width} ${leg3_width} ${leg3_height-leg3_tip_radius}"/>
+        </geometry>
       <material name="Red"/>
     </collision>
     <collision>
-      <origin xyz="0 ${revert*leg3_length-revert*leg3_tip_radius} ${leg3_dist}"
+      <origin xyz="0 ${leg3_length-leg3_width/2} -${leg3_height}"
         rpy="${PI_2} 0 0"/>
             <geometry>

File: hexapod_description/urdf/modules/leg_marta.xacro (robot description, xacro)
@@ -7,26 +7,28 @@
             <child link="leg_${index}_1"/>
             <limit effort="${joint_eff}" lower="${-joint_lim}" upper="${joint_lim}" velocity="${joint_vel}"/>
-            <xacro:if value="${index == 5 or index == 2}">
-                <origin rpy="0 0 -0.3" xyz="${xPos} ${yPos} 0"/>
+            <!-- Add a small offset angle to match the default position on the robot -->
+            <xacro:if value="${(index+1) % 3 == 0}">
+                <xacro:property name="offset_angle" value= "-0.3"/>
             </xacro:if>
-            <xacro:if value="${index == 0 or index == 3}">
-                <origin rpy="0 0 0.3" xyz="${xPos} ${yPos} 0"/>
+            <xacro:if value="${(index+1) % 3 == 1}">
+                <xacro:property name="offset_angle" value= "0.3"/>
             </xacro:if>
-            <xacro:if value="${index == 1 or index == 4}">
-                <origin rpy="0 0 0" xyz="${xPos} ${yPos} 0"/>
+            <xacro:if value="${(index+1) % 3 == 2}">
+                <xacro:property name="offset_angle" value= "0"/>
             </xacro:if>
-            <!-- <xacro:if value="${index == 5 or index == 4 or index == 3}">
-                <axis xyz="0 0 1"/>
+            <!-- Angle for the legs of the left side -->
+            <xacro:property name="legs_rotation" value="0"/>
+            <xacro:if value="${index > 2}">
+                <xacro:property name="legs_rotation" value="${PI}"/>
             </xacro:if>
-            <xacro:if value="${index == 2 or index == 1 or index == 0}"> -->
-                <axis xyz="0 0 1"/>
-            <!-- </xacro:if> -->
+            <origin rpy="0 0 ${offset_angle+legs_rotation}" xyz="${xPos} ${yPos} 0"/>
+            <axis xyz="0 0 1"/>
             <dynamics damping="${joint_dmp}"/>
         </joint>
         <link name="leg_${index}_1">
-            <xacro:visuals_collisions_leg_1 revert="${sign}"/>
+            <xacro:visuals_collisions_leg_1/>
             <inertial>
                 <!-- CENTER OF MASS -->
-                <origin rpy="${PI_2} 0 0" xyz="${leg1_width/2} ${sign*leg1_length/2} 0"/>
+                <origin rpy="${PI_2} 0 0" xyz="${leg1_width/2} ${leg1_length/2} 0"/>
                 <mass value="${leg1_mass}"/>
                 <!-- box inertia: 1/12*m(y^2+z^2), ... -->
@@ -38,18 +40,13 @@
             <child link="leg_${index}_2"/>
             <limit effort="${joint_eff}" lower="${-joint_lim}" upper="${joint_lim}" velocity="${joint_vel}"/>
-            <origin rpy="0 0 0" xyz="0 ${sign*leg1_length} 0"/>
-            <xacro:if value="${index == 5 or index == 4 or index == 3}">
-                <axis xyz="-1 0 0"/>
-            </xacro:if>
-            <xacro:if value="${index == 2 or index == 1 or index == 0}">
-                <axis xyz="1 0 0"/>
-            </xacro:if>
+            <origin rpy="0 0 0" xyz="0 ${leg1_length} 0"/>
+            <axis xyz="1 0 0"/>
             <dynamics damping="${joint_dmp}"/>
         </joint>
         <link name="leg_${index}_2">
-            <xacro:visuals_collisions_leg_2 revert="${sign}"/>
+            <xacro:visuals_collisions_leg_2/>
             <inertial>
                 <!-- CENTER OF MASS -->
-                <origin rpy="${PI_2} 0 0" xyz="${leg2_width/2} ${sign*leg2_length/2} 0"/>
+                <origin rpy="${PI_2} 0 0" xyz="${leg2_width/2} ${leg2_length/2} 0"/>
                 <mass value="${leg2_mass}"/>
                 <!-- box inertia: 1/12*m(y^2+z^2), ... -->
@@ -61,18 +58,13 @@
             <child link="leg_${index}_3"/>
             <limit effort="${joint_eff}" lower="${-joint_lim}" upper="${joint_lim}" velocity="${joint_vel}"/>
-            <origin rpy="${-sign*PI_2} 0 0" xyz="0 ${sign*leg2_length} 0"/>
-            <xacro:if value="${index == 5 or index == 4 or index == 3}">
-                <axis xyz="1 0 0"/>
-            </xacro:if>
-            <xacro:if value="${index == 2 or index == 1 or index == 0}">
-                <axis xyz="-1 0 0"/>
-            </xacro:if>
+            <origin rpy="0 0 0" xyz="0 ${leg2_length} 0"/>
+            <axis xyz="1 0 0"/>
             <dynamics damping="${joint_dmp}"/>
         </joint>
         <link name="leg_${index}_3">
-            <xacro:visuals_collisions_leg_3 revert="${sign}"/>
+            <xacro:visuals_collisions_leg_3/>
             <inertial>
                 <!-- CENTER OF MASS -->
-                <origin rpy="${PI_2} 0 0" xyz="0 ${sign*leg3_length/2} 0"/>
+                <origin rpy="${PI_2} 0 0" xyz="0 ${leg3_length/2} 0"/>
                 <mass value="${leg3_mass}"/>
                 <!-- box inertia: 1/12*m(y^2+z^2), ... -->
@@ -83,7 +75,8 @@
             <parent link="leg_${index}_3"/>
             <child link="force_sensor_${index}"/>
-            <origin rpy="${-sign*PI_2} 0 0" xyz="0 ${sign*leg3_length} ${leg3_dist}"/>
+            <origin rpy="${PI} 0 ${PI_2}" xyz="0 ${force_y_offset} -${force_z_offset}"/>
         </joint>
         <link name="force_sensor_${index}"/>
+        <!-- Description used by our Dart simulator -->
         <dart_sensor type="force">
           <link>force_sensor_${index}</link>

File: hexapod_description/urdf/modules/marta.xacro (robot description, xacro)
@@ -9,5 +9,5 @@
   <xacro:property name="body_length" value="0.24"/>
   <xacro:property name="body_width" value="0.119"/>
-  <xacro:property name="body_width_extra" value="0.190"/>
+  <xacro:property name="body_width_extra" value="0.199"/>
   <xacro:property name="body_height" value="0.04"/>
   <xacro:property name="leg1_width" value="0.05"/>
@@ -20,8 +20,11 @@
   <xacro:property name="leg2_mass" value="0.184"/>
   <xacro:property name="leg3_width" value="0.054"/>
-  <xacro:property name="leg3_length" value="0.12"/>
-  <xacro:property name="leg3_dist" value="0.038"/>
+  <xacro:property name="leg3_length" value="0.065"/>
+  <xacro:property name="leg3_dist" value="0.032"/>
+  <xacro:property name="leg3_height" value="0.10"/>
   <xacro:property name="leg3_tip_radius" value="0.02"/>
   <xacro:property name="leg3_mass" value="0.04"/>
+  <xacro:property name="force_y_offset" value="${(11.25+27)*0.001}"/>
+  <xacro:property name="force_z_offset" value="0.115"/>
   <xacro:property name="joint_lim" value="${PI_2}"/>
   <xacro:property name="joint_eff" value="30.0"/>
