Commit message: Update the model for Pexod, the same way as was done for Hexaforce

File: hexapod_description/urdf/hexaforce_visuals_collisions.xacro (robot description, xacro)
@@ -83,10 +83,10 @@
       <origin xyz="0 0 0" rpy="0 0 ${PI}"/>
       <geometry>
-        <mesh filename="package://hexapod_description/stl/third_link.stl" scale="0.001 0.001 0.001"/>
+        <mesh filename="package://hexapod_description/stl/third_link_v5.stl" scale="0.001 0.001 0.001"/>
         <material name="Red"/>
       </geometry>
     </visual>
     <collision>
-      <origin xyz="0 ${leg3_dist} 0" rpy="0 0 0"/>
+      <origin xyz="0 ${leg3_length/2} 0" rpy="0 0 0"/>
         <geometry>
           <box size="${leg3_width} ${leg3_length} ${leg3_width}"/>

File: hexapod_description/urdf/modules/hexaforce.xacro (robot description, xacro)
@@ -21,5 +21,4 @@
   <xacro:property name="leg3_width" value="0.054"/>
   <xacro:property name="leg3_length" value="0.065"/>
-  <xacro:property name="leg3_dist" value="0.032"/>
   <xacro:property name="leg3_height" value="0.10"/>
   <xacro:property name="leg3_tip_radius" value="0.02"/>

File: hexapod_description/urdf/modules/leg_hexaforce.xacro (robot description, xacro)
@@ -2,5 +2,5 @@
 <robot xmlns:xacro="http://www.ros.org/wiki/xacro">
   <!-- XACRO MACRO FOR LEGS LINKS/JOINTS -->
-    <xacro:macro name="leg" params="index xPos yPos sign">
+    <xacro:macro name="leg" params="index xPos yPos">
         <joint name="body_leg_${index}" type="revolute">
             <parent link="base_link"/>

File: hexapod_description/urdf/modules/leg_pexod.xacro (robot description, xacro)
@@ -2,31 +2,33 @@
 <robot xmlns:xacro="http://www.ros.org/wiki/xacro">
   <!-- XACRO MACRO FOR LEGS LINKS/JOINTS -->
-    <xacro:macro name="leg" params="index xPos yPos sign">
+    <xacro:macro name="leg" params="index xPos yPos">
         <joint name="body_leg_${index}" type="revolute">
             <parent link="base_link"/>
             <child link="leg_${index}_1"/>
             <limit effort="${joint_eff}" lower="${-joint_lim}" upper="${joint_lim}" velocity="${joint_vel}"/>
-            <xacro:if value="${index == 5 or index == 2}">
-                <origin rpy="0 0 -0.3" xyz="${xPos} ${yPos} 0"/>
+            <!-- Add a small offset angle to match the default position on the robot -->
+            <xacro:if value="${(index+1) % 3 == 0}">
+                <xacro:property name="offset_angle" value= "-0.3"/>
             </xacro:if>
-            <xacro:if value="${index == 0 or index == 3}">
-                <origin rpy="0 0 0.3" xyz="${xPos} ${yPos} 0"/>
+            <xacro:if value="${(index+1) % 3 == 1}">
+                <xacro:property name="offset_angle" value= "0.3"/>
             </xacro:if>
-            <xacro:if value="${index == 1 or index == 4}">
-                <origin rpy="0 0 0" xyz="${xPos} ${yPos} 0"/>
+            <xacro:if value="${(index+1) % 3 == 2}">
+                <xacro:property name="offset_angle" value= "0"/>
             </xacro:if>
-            <!-- <xacro:if value="${index == 5 or index == 4 or index == 3}">
-                <axis xyz="0 0 1"/>
+            <!-- Angle for the legs of the left side -->
+            <xacro:property name="legs_rotation" value="0"/>
+            <xacro:if value="${index > 2}">
+                <xacro:property name="legs_rotation" value="${PI}"/>
             </xacro:if>
-            <xacro:if value="${index == 2 or index == 1 or index == 0}"> -->
-                <axis xyz="0 0 1"/>
-            <!-- </xacro:if> -->
+            <origin rpy="0 0 ${offset_angle+legs_rotation}" xyz="${xPos} ${yPos} 0"/>
+            <axis xyz="0 0 1"/>
             <dynamics damping="${joint_dmp}"/>
         </joint>
         <link name="leg_${index}_1">
-            <xacro:visuals_collisions_leg_1 revert="${sign}"/>
+            <xacro:visuals_collisions_leg_1/>
             <inertial>
                 <!-- CENTER OF MASS -->
-                <origin rpy="${PI_2} 0 0" xyz="${leg1_width/2} ${sign*leg1_length/2} 0"/>
+                <origin rpy="${PI_2} 0 0" xyz="${leg1_width/2} ${leg1_length/2} 0"/>
                 <mass value="${leg1_mass}"/>
                 <!-- box inertia: 1/12*m(y^2+z^2), ... -->
@@ -38,18 +40,13 @@
             <child link="leg_${index}_2"/>
             <limit effort="${joint_eff}" lower="${-joint_lim2}" upper="${joint_lim2}" velocity="${joint_vel}"/>
-            <origin rpy="0 0 0" xyz="0 ${sign*leg1_length} 0"/>
-            <xacro:if value="${index == 5 or index == 4 or index == 3}">
-                <axis xyz="-1 0 0"/>
-            </xacro:if>
-            <xacro:if value="${index == 2 or index == 1 or index == 0}">
-                <axis xyz="1 0 0"/>
-            </xacro:if>
+            <origin rpy="0 0 0" xyz="0 ${leg1_length} 0"/>
+            <axis xyz="1 0 0"/>
             <dynamics damping="${joint_dmp}"/>
         </joint>
         <link name="leg_${index}_2">
-            <xacro:visuals_collisions_leg_2 revert="${sign}"/>
+            <xacro:visuals_collisions_leg_2/>
             <inertial>
                 <!-- CENTER OF MASS -->
-                <origin rpy="${PI_2} 0 0" xyz="${leg2_width/2} ${sign*leg2_length/2} 0"/>
+                <origin rpy="${PI_2} 0 0" xyz="${leg2_width/2} ${leg2_length/2} 0"/>
                 <mass value="${leg2_mass}"/>
                 <!-- box inertia: 1/12*m(y^2+z^2), ... -->
@@ -61,18 +58,13 @@
             <child link="leg_${index}_3"/>
             <limit effort="${joint_eff}" lower="${-joint_lim2}" upper="${joint_lim2}" velocity="${joint_vel}"/>
-            <origin rpy="${-sign*PI_2} 0 0" xyz="0 ${sign*leg2_length} 0"/>
-            <xacro:if value="${index == 5 or index == 4 or index == 3}">
-                <axis xyz="1 0 0"/>
-            </xacro:if>
-            <xacro:if value="${index == 2 or index == 1 or index == 0}">
-                <axis xyz="-1 0 0"/>
-            </xacro:if>
+            <origin rpy="${PI_2} 0 0" xyz="0 ${leg2_length} 0"/>
+            <axis xyz="1 0 0"/>
             <dynamics damping="${joint_dmp}"/>
         </joint>
         <link name="leg_${index}_3">
-            <xacro:visuals_collisions_leg_3 revert="${sign}"/>
+            <xacro:visuals_collisions_leg_3/>
             <inertial>
                 <!-- CENTER OF MASS -->
-                <origin rpy="${PI_2} 0 0" xyz="0 ${sign*leg3_length/2} 0"/>
+                <origin rpy="${PI_2} 0 0" xyz="0 ${leg3_length/2} 0"/>
                 <mass value="${leg3_mass}"/>
                 <!-- box inertia: 1/12*m(y^2+z^2), ... -->

File: hexapod_description/urdf/modules/legs_hexaforce.xacro (robot description, xacro)
@@ -2,10 +2,10 @@
 <robot xmlns:xacro="http://www.ros.org/wiki/xacro">
   <!-- LEGS LINKS/JOINTS -->
-    <xacro:leg index="2" xPos="${body_length/2}" yPos="${body_width/2}" sign="1"/>
-    <xacro:leg index="3" xPos="${body_length/2}" yPos="${-body_width/2}" sign="-1"/>
-    <xacro:leg index="0" xPos="${-body_length/2}" yPos="${body_width/2}" sign="1"/>
-    <xacro:leg index="5" xPos="${-body_length/2}" yPos="${-body_width/2}" sign="-1"/>
-    <xacro:leg index="1" xPos="0" yPos="${body_width_extra/2}" sign="1"/>
-    <xacro:leg index="4" xPos="0" yPos="${-body_width_extra/2}" sign="-1"/>
+    <xacro:leg index="2" xPos="${body_length/2}" yPos="${body_width/2}"/>
+    <xacro:leg index="3" xPos="${body_length/2}" yPos="${-body_width/2}"/>
+    <xacro:leg index="0" xPos="${-body_length/2}" yPos="${body_width/2}"/>
+    <xacro:leg index="5" xPos="${-body_length/2}" yPos="${-body_width/2}"/>
+    <xacro:leg index="1" xPos="0" yPos="${body_width_extra/2}"/>
+    <xacro:leg index="4" xPos="0" yPos="${-body_width_extra/2}"/>
   <!-- END OF LEG LINKS/JOINTS -->
 </robot>

File: hexapod_description/urdf/modules/pexod.xacro (robot description, xacro)
@@ -9,16 +9,19 @@
   <xacro:property name="body_length" value="0.24"/>
   <xacro:property name="body_width" value="0.119"/>
-  <xacro:property name="body_width_extra" value="0.190"/>
+  <xacro:property name="body_width_extra" value="0.199"/>
   <xacro:property name="body_height" value="0.04"/>
-  <xacro:property name="leg1_width" value="0.02"/>
+  <xacro:property name="leg1_width" value="0.044"/>
   <xacro:property name="leg1_length" value="0.06"/>
   <xacro:property name="leg1_dist" value="0.2"/>
   <xacro:property name="leg1_mass" value="0.02"/>
-  <xacro:property name="leg2_width" value="0.02"/>
+  <xacro:property name="leg2_width" value="0.038"/>
   <xacro:property name="leg2_length" value="0.0835"/>
   <xacro:property name="leg2_dist" value="0.2"/>
   <xacro:property name="leg2_mass" value="0.184"/>
-  <xacro:property name="leg3_width" value="0.025"/>
-  <xacro:property name="leg3_length" value="0.140"/>
+  <xacro:property name="leg3_width" value="0.052"/>
+  <xacro:property name="leg3_width2" value="0.022"/>
+  <xacro:property name="leg3_length" value="0.053"/>
+  <xacro:property name="leg3_height" value="0.142"/>
+  <xacro:property name="leg3_tip_radius" value="0.02"/>
   <xacro:property name="leg3_mass" value="0.04"/>
   <xacro:property name="joint_lim" value="${PI_2}"/>

File: hexapod_description/urdf/pexod_visuals_collisions.xacro (robot description, xacro)
@@ -21,16 +21,9 @@
     <xacro:macro name="visuals_collisions_body" params="">
     <visual>
-      <origin xyz="0 0 0" rpy="0 0 0"/>
-            <geometry>
-                <box size="${body_length} ${body_width} ${body_height}"/>
-            </geometry>
-      <material name="LightGrey"/>
-    </visual>
-    <visual>
-      <origin xyz="0 0 0" rpy="0 0 0"/>
-            <geometry>
-                <box size="${leg1_width*2.5} ${body_width_extra} ${body_height}"/>
-            </geometry>
-      <material name="LightGrey"/>
+      <origin xyz="0 0 0" rpy="${PI_2} 0 ${PI_2}"/>
+        <geometry>
+          <mesh filename="package://hexapod_description/stl/chassis.stl" scale="0.001 0.001 0.001"/>
+        </geometry>
+      <material name="Yellow"/>
     </visual>
     <collision>
@@ -49,66 +42,76 @@
   <xacro:macro name="visuals_head" params="">
     <visual>
-      <origin xyz="${body_length/2.} 0 ${body_height*0.7}" rpy="0 0 ${PI/4}"/>
+      <origin xyz="${body_length/2.} 0 0" rpy="0 0 ${PI/4}"/>
       <geometry>
-        <box size="${body_width/2.} ${body_width/2.} ${body_height*0.7}"/>
+        <box size="${body_width/3.} ${body_width/3.} ${body_height*0.6}"/>
       </geometry>
       <material name="Yellow"/>
     </visual>
   </xacro:macro>
-  <xacro:macro name="visuals_collisions_leg_1" params="revert">
+  <xacro:macro name="visuals_collisions_leg_1">
     <visual>
-      <origin xyz="0 ${revert*leg1_length/2} 0" rpy="${PI_2} 0 0"/>
-            <geometry>
-                <cylinder radius="${leg1_width}" length="${leg1_length}"/>
-            </geometry>
+      <origin xyz="0 0 0" rpy="0 ${PI_2} 0"/>
+        <geometry>
+          <mesh filename="package://hexapod_description/stl/first_link.stl" scale="0.001 0.001 0.001"/>
+        </geometry>
       <material name="Red"/>
     </visual>
     <collision>
-      <origin xyz="0 ${revert*leg1_length/2} 0" rpy="${PI_2} 0 0"/>
-            <geometry>
-                <box size="${leg1_width} ${leg1_width} ${leg1_length}"/>
-            </geometry>
+      <origin xyz="0 ${leg1_length/2} 0" rpy="${PI_2} 0 0"/>
+        <geometry>
+          <box size="${leg1_width} ${leg1_width} ${leg1_length}"/>
+        </geometry>
     </collision>
   </xacro:macro>
-  <xacro:macro name="visuals_collisions_leg_2" params="revert">
+  <xacro:macro name="visuals_collisions_leg_2">
     <visual>
-      <origin xyz="0 ${revert*leg2_length/2} 0" rpy="${PI_2} 0 0"/>
-            <geometry>
-                <cylinder radius="${leg2_width}" length="${leg2_length}"/>
-            </geometry>
+      <origin xyz="0 0 0" rpy="0 -${PI_2} 0"/>
+        <geometry>
+          <mesh filename="package://hexapod_description/stl/second_link.stl" scale="0.001 0.001 0.001"/>
+        </geometry>
       <material name="Blue"/>
     </visual>
     <collision>
-      <origin xyz="0 ${revert*leg2_length/2} 0" rpy="${PI_2} 0 0"/>
-            <geometry>
-                <box size="${leg2_width} ${leg2_width} ${leg2_length}"/>
-            </geometry>
+      <origin xyz="0 ${leg2_length/2} 0" rpy="${PI_2} 0 0"/>
+        <geometry>
+          <box size="${leg2_width} ${leg2_width} ${leg2_length}"/>
+        </geometry>
     </collision>
   </xacro:macro>
-  <xacro:macro name="visuals_collisions_leg_3" params="revert">
+  <xacro:macro name="visuals_collisions_leg_3">
     <visual>
-      <origin xyz="0 ${revert*leg3_length/2} 0" rpy="${PI_2} 0 0"/>
-            <geometry>
-              <cylinder radius="${leg3_width}" length="${leg3_length}"/>
-            </geometry>
-      <material name="Red"/>
+      <origin xyz="0 0 0" rpy="${-PI_2} 0 0"/>
+      <geometry>
+        <mesh filename="package://hexapod_description/stl/FR07-H101-centered.stl" scale="0.001 0.001 0.001"/>
+        <material name="Red"/>
+      </geometry>
     </visual>
     <visual>
-      <origin xyz="0 ${revert*leg3_length-revert*leg3_width/2} 0" rpy="${PI_2} 0 0"/>
-            <geometry>
-                <sphere radius="${leg3_width}"/>
-            </geometry>
-      <material name="Red"/>
+      <origin xyz="0 0 -0.03" rpy="0 0 ${PI}"/>
+      <geometry>
+        <mesh filename="package://hexapod_description/stl/third_link_v4.stl" scale="0.001 0.001 0.001"/>
+        <material name="Red"/>
+      </geometry>
     </visual>
     <collision>
-      <origin xyz="0 ${revert*leg3_length/2} 0" rpy="${PI_2} 0 0"/>
-            <geometry>
-                <box size="${leg3_width} ${leg3_width} ${leg3_length}"/>
-            </geometry>
+      <origin xyz="0 0 -${leg3_length/2}" rpy="0 0 0"/>
+        <geometry>
+          <box size="${leg3_width} ${leg3_width} ${leg3_length}"/>
+        </geometry>
+      <material name="Red"/>
     </collision>
     <collision>
-      <origin xyz="0 ${revert*leg3_length-revert*leg3_width/2} 0" rpy="${PI_2} 0 0"/>
+      <origin xyz="0 ${leg3_length-leg3_width/2} ${-(leg3_height-leg3_tip_radius)/2}"
+        rpy="0 0 0"/>
+        <geometry>
+          <box size="${leg3_width} ${leg3_width2} ${leg3_height-leg3_tip_radius}"/>
+        </geometry>
+      <material name="Red"/>
+    </collision>
+    <collision>
+      <origin xyz="0 ${leg3_length-leg3_width/2} -${leg3_height-leg3_tip_radius}"
+        rpy="${PI_2} 0 0"/>
             <geometry>
-                <sphere radius="${leg3_width}"/>
+                <sphere radius="${leg3_tip_radius}"/>
             </geometry>
       <material name="Red"/>

Commit message: Minor fix for material

File: hexapod_description/urdf/hexaforce_visuals_collisions.xacro (robot description, xacro)
@@ -84,6 +84,6 @@
       <geometry>
         <mesh filename="package://hexapod_description/stl/third_link_v5.stl" scale="0.001 0.001 0.001"/>
-        <material name="Red"/>
       </geometry>
+      <material name="Red"/>
     </visual>
     <collision>

Commit message: Update for latest version of Pexod

File: hexapod_description/urdf/hexaforce_visuals_collisions.xacro (robot description, xacro)
@@ -15,9 +15,9 @@
   </material>
   <material name="LightGrey">
-      <color rgba="0.6 0.6 0.6 1.0"/>
+    <color rgba="0.6 0.6 0.6 1.0"/>
   </material>
-    <!-- END OF MATERIALS -->
-    <!-- XACRO MACROS FOR VISUALS AND COLLISIONS -->
-    <xacro:macro name="visuals_collisions_body" params="">
+  <!-- END OF MATERIALS -->
+  <!-- XACRO MACROS FOR VISUALS AND COLLISIONS -->
+  <xacro:macro name="visuals_collisions_body" params="">
     <visual>
       <origin xyz="0 0 0" rpy="${PI_2} 0 ${PI_2}"/>

File: hexapod_description/urdf/modules/leg_hexaforce.xacro (robot description, xacro)
@@ -1,5 +1,5 @@
 <?xml version="1.0"?>
 <robot xmlns:xacro="http://www.ros.org/wiki/xacro">
-  <!-- XACRO MACRO FOR LEGS LINKS/JOINTS -->
+    <!-- XACRO MACRO FOR LEGS LINKS/JOINTS -->
     <xacro:macro name="leg" params="index xPos yPos">
         <joint name="body_leg_${index}" type="revolute">

File: hexapod_description/urdf/modules/leg_pexod.xacro (robot description, xacro)
@@ -39,5 +39,5 @@
             <parent link="leg_${index}_1"/>
             <child link="leg_${index}_2"/>
-            <limit effort="${joint_eff}" lower="${-joint_lim2}" upper="${joint_lim2}" velocity="${joint_vel}"/>
+            <limit effort="${joint_eff}" lower="${-joint_lim}" upper="${joint_lim}" velocity="${joint_vel}"/>
             <origin rpy="0 0 0" xyz="0 ${leg1_length} 0"/>
             <axis xyz="1 0 0"/>
@@ -57,5 +57,5 @@
             <parent link="leg_${index}_2"/>
             <child link="leg_${index}_3"/>
-            <limit effort="${joint_eff}" lower="${-joint_lim2}" upper="${joint_lim2}" velocity="${joint_vel}"/>
+            <limit effort="${joint_eff}" lower="${-joint_lim}" upper="${joint_lim}" velocity="${joint_vel}"/>
             <origin rpy="0 0 0" xyz="0 ${leg2_length} 0"/>
             <axis xyz="-1 0 0"/>

File: hexapod_description/urdf/modules/pexod.xacro (robot description, xacro)
@@ -19,12 +19,10 @@
   <xacro:property name="leg2_dist" value="0.2"/>
   <xacro:property name="leg2_mass" value="0.184"/>
-  <xacro:property name="leg3_width" value="0.052"/>
-  <xacro:property name="leg3_width2" value="0.022"/>
-  <xacro:property name="leg3_length" value="0.053"/>
-  <xacro:property name="leg3_height" value="0.142"/>
+  <xacro:property name="leg3_width" value="0.054"/>
+  <xacro:property name="leg3_length" value="0.065"/>
+  <xacro:property name="leg3_height" value="0.10"/>
   <xacro:property name="leg3_tip_radius" value="0.02"/>
   <xacro:property name="leg3_mass" value="0.04"/>
   <xacro:property name="joint_lim" value="${PI_2}"/>
-  <xacro:property name="joint_lim2" value="${PI_4}"/>
   <xacro:property name="joint_eff" value="30.0"/>
   <xacro:property name="joint_vel" value="7.0"/>

File: hexapod_description/urdf/pexod_visuals_collisions.xacro (robot description, xacro)
@@ -12,12 +12,12 @@
   </material>
   <material name="Yellow">
-    <color rgba="1 1 0 1"/>
-    </material>
-    <material name="LightGrey">
-      <color rgba="0.5 0.5 0.85 1.0"/>
+    <color rgba="0.8 0.9 0.3 1"/>
   </material>
-    <!-- END OF MATERIALS -->
-    <!-- XACRO MACROS FOR VISUALS AND COLLISIONS -->
-    <xacro:macro name="visuals_collisions_body" params="">
+  <material name="LightGrey">
+    <color rgba="0.6 0.6 0.6 1.0"/>
+  </material>
+  <!-- END OF MATERIALS -->
+  <!-- XACRO MACROS FOR VISUALS AND COLLISIONS -->
+  <xacro:macro name="visuals_collisions_body" params="">
     <visual>
       <origin xyz="0 0 0" rpy="${PI_2} 0 ${PI_2}"/>
@@ -81,34 +81,27 @@
   <xacro:macro name="visuals_collisions_leg_3">
     <visual>
-      <origin xyz="0 0 0" rpy="${-PI_2} 0 0"/>
+      <origin xyz="0 0 0" rpy="0 0 ${PI}"/>
       <geometry>
-        <mesh filename="package://hexapod_description/stl/FR07-H101-centered.stl" scale="0.001 0.001 0.001"/>
-        <material name="Red"/>
+        <mesh filename="package://hexapod_description/stl/third_link_v4.5.stl" scale="0.001 0.001 0.001"/>
       </geometry>
-    </visual>
-    <visual>
-      <origin xyz="0 0 -0.03" rpy="0 0 ${PI}"/>
-      <geometry>
-        <mesh filename="package://hexapod_description/stl/third_link_v4.stl" scale="0.001 0.001 0.001"/>
-        <material name="Red"/>
-      </geometry>
+      <material name="Red"/>
     </visual>
     <collision>
-      <origin xyz="0 0 -${leg3_length/2}" rpy="0 0 0"/>
+      <origin xyz="0 ${leg3_length/2} 0" rpy="0 0 0"/>
         <geometry>
-          <box size="${leg3_width} ${leg3_width} ${leg3_length}"/>
+          <box size="${leg3_width} ${leg3_length} ${leg3_width}"/>
         </geometry>
       <material name="Red"/>
     </collision>
     <collision>
-      <origin xyz="0 ${leg3_length-leg3_width/2} ${-(leg3_height-leg3_tip_radius)/2}"
+      <origin xyz="0 ${leg3_length-leg3_width/2} ${-(leg3_width+leg3_height-leg3_tip_radius)/2}"
         rpy="0 0 0"/>
         <geometry>
-          <box size="${leg3_width} ${leg3_width2} ${leg3_height-leg3_tip_radius}"/>
+          <box size="${leg3_width} ${leg3_width} ${leg3_height-leg3_tip_radius}"/>
         </geometry>
       <material name="Red"/>
     </collision>
     <collision>
-      <origin xyz="0 ${leg3_length-leg3_width/2} -${leg3_height-leg3_tip_radius}"
+      <origin xyz="0 ${leg3_length-leg3_width/2} -${leg3_height}"
         rpy="${PI_2} 0 0"/>
             <geometry>
