Commit message: tinkering with URDF generation

File: hexapod_description/urdf/hexaforce.xacro (robot description, xacro)
@@ -1,4 +1,11 @@
 <?xml version="1.0"?>
 <robot name="pexod" xmlns:xacro="http://www.ros.org/wiki/xacro">
+  <xacro:property name="path_generation" value="relative" />
+  <xacro:if value="${'package' == path_generation}">
+    <xacro:property name="path_prefix" value="package://hexapod_description/" />
+  </xacro:if>
+  <xacro:if value="${'relative' == path_generation}">
+    <xacro:property name="path_prefix" value="" />
+  </xacro:if>
   <xacro:include filename="$(find hexapod_description)/urdf/modules/hexaforce.xacro" />
 </robot>

File: hexapod_description/urdf/hexaforce_visuals_collisions.xacro (robot description, xacro)
@@ -23,5 +23,6 @@
       <origin xyz="0 0 0" rpy="${PI_2} 0 ${PI_2}"/>
         <geometry>
-          <mesh filename="package://hexapod_description/stl/chassis.stl" scale="0.001 0.001 0.001"/>
+          <!-- <mesh filename="${path_prefix}" scale="0.001 0.001 0.001"/> -->
+          <mesh filename="${path_prefix + 'stl/chassis.stl'}" scale="0.001 0.001 0.001"/>
         </geometry>
       <material name="Yellow"/>

Commit message: generate ROS-dependant/independant versions of URDF

File: hexapod_description/urdf/hexaforce.xacro (robot description, xacro)
@@ -1,10 +1,11 @@
 <?xml version="1.0"?>
 <robot name="pexod" xmlns:xacro="http://www.ros.org/wiki/xacro">
-  <xacro:property name="path_generation" value="relative" />
+  <xacro:arg name="path_generation" default="package" />
+  <xacro:property name="path_generation" value="$(arg path_generation)" />
   <xacro:if value="${'package' == path_generation}">
     <xacro:property name="path_prefix" value="package://hexapod_description/" />
   </xacro:if>
   <xacro:if value="${'relative' == path_generation}">
-    <xacro:property name="path_prefix" value="" />
+    <xacro:property name="path_prefix" value="../" />
   </xacro:if>
   <xacro:include filename="$(find hexapod_description)/urdf/modules/hexaforce.xacro" />

File: hexapod_description/urdf/hexaforce_visuals_collisions.xacro (robot description, xacro)
@@ -23,5 +23,4 @@
       <origin xyz="0 0 0" rpy="${PI_2} 0 ${PI_2}"/>
         <geometry>
-          <!-- <mesh filename="${path_prefix}" scale="0.001 0.001 0.001"/> -->
           <mesh filename="${path_prefix + 'stl/chassis.stl'}" scale="0.001 0.001 0.001"/>
         </geometry>
@@ -54,5 +53,5 @@
       <origin xyz="0 0 0" rpy="0 ${PI_2} 0"/>
         <geometry>
-          <mesh filename="package://hexapod_description/stl/first_link.stl" scale="0.001 0.001 0.001"/>
+          <mesh filename="${path_prefix + 'stl/first_link.stl'}" scale="0.001 0.001 0.001"/>
         </geometry>
       <material name="Red"/>
@@ -69,5 +68,5 @@
       <origin xyz="0 0 0" rpy="0 -${PI_2} 0"/>
         <geometry>
-          <mesh filename="package://hexapod_description/stl/second_link.stl" scale="0.001 0.001 0.001"/>
+          <mesh filename="${path_prefix + 'stl/second_link.stl'}" scale="0.001 0.001 0.001"/>
         </geometry>
       <material name="Blue"/>
@@ -84,5 +83,5 @@
       <origin xyz="0 0 0" rpy="0 0 ${PI}"/>
       <geometry>
-        <mesh filename="package://hexapod_description/stl/third_link_v5.stl" scale="0.001 0.001 0.001"/>
+        <mesh filename="${path_prefix + 'stl/third_link_v5.stl'}" scale="0.001 0.001 0.001"/>
       </geometry>
       <material name="Red"/>

File: hexapod_description/urdf/pexod.xacro (robot description, xacro)
@@ -1,4 +1,12 @@
 <?xml version="1.0"?>
 <robot name="pexod" xmlns:xacro="http://www.ros.org/wiki/xacro">
+  <xacro:arg name="path_generation" default="package" />
+  <xacro:property name="path_generation" value="$(arg path_generation)" />
+  <xacro:if value="${'package' == path_generation}">
+    <xacro:property name="path_prefix" value="package://hexapod_description/" />
+  </xacro:if>
+  <xacro:if value="${'relative' == path_generation}">
+    <xacro:property name="path_prefix" value="../" />
+  </xacro:if>
   <xacro:include filename="$(find hexapod_description)/urdf/modules/pexod.xacro" />
 </robot>

File: hexapod_description/urdf/pexod_visuals_collisions.xacro (robot description, xacro)
@@ -23,5 +23,5 @@
       <origin xyz="0 0 0" rpy="${PI_2} 0 ${PI_2}"/>
         <geometry>
-          <mesh filename="package://hexapod_description/stl/chassis.stl" scale="0.001 0.001 0.001"/>
+          <mesh filename="${path_prefix + 'stl/chassis.stl'}" scale="0.001 0.001 0.001"/>
         </geometry>
       <material name="Yellow"/>
@@ -53,5 +53,5 @@
       <origin xyz="0 0 0" rpy="0 ${PI_2} 0"/>
         <geometry>
-          <mesh filename="package://hexapod_description/stl/first_link.stl" scale="0.001 0.001 0.001"/>
+          <mesh filename="${path_prefix + 'stl/first_link.stl'}" scale="0.001 0.001 0.001"/>
         </geometry>
       <material name="Red"/>
@@ -68,5 +68,5 @@
       <origin xyz="0 0 0" rpy="0 -${PI_2} 0"/>
         <geometry>
-          <mesh filename="package://hexapod_description/stl/second_link.stl" scale="0.001 0.001 0.001"/>
+          <mesh filename="${path_prefix + 'stl/second_link.stl'}" scale="0.001 0.001 0.001"/>
         </geometry>
       <material name="Blue"/>
@@ -83,5 +83,5 @@
       <origin xyz="0 0 0" rpy="0 0 ${PI}"/>
       <geometry>
-        <mesh filename="package://hexapod_description/stl/third_link_v4.5.stl" scale="0.001 0.001 0.001"/>
+        <mesh filename="${path_prefix + 'stl/third_link_v4.5.stl'}" scale="0.001 0.001 0.001"/>
       </geometry>
       <material name="Red"/>

Commit message: Change location of generated URDFs for simulation

File: hexapod_description/urdf/hexaforce.xacro (robot description, xacro)
@@ -7,5 +7,5 @@
   </xacro:if>
   <xacro:if value="${'relative' == path_generation}">
-    <xacro:property name="path_prefix" value="../" />
+    <xacro:property name="path_prefix" value="" />
   </xacro:if>
   <xacro:include filename="$(find hexapod_description)/urdf/modules/hexaforce.xacro" />

File: hexapod_description/urdf/pexod.xacro (robot description, xacro)
@@ -7,5 +7,5 @@
   </xacro:if>
   <xacro:if value="${'relative' == path_generation}">
-    <xacro:property name="path_prefix" value="../" />
+    <xacro:property name="path_prefix" value="" />
   </xacro:if>
   <xacro:include filename="$(find hexapod_description)/urdf/modules/pexod.xacro" />

Commit message: Better relative path and generating ROS urdfs also

File: hexapod_description/urdf/hexaforce.xacro (robot description, xacro)
@@ -7,5 +7,5 @@
   </xacro:if>
   <xacro:if value="${'relative' == path_generation}">
-    <xacro:property name="path_prefix" value="" />
+    <xacro:property name="path_prefix" value="./" />
   </xacro:if>
   <xacro:include filename="$(find hexapod_description)/urdf/modules/hexaforce.xacro" />

File: hexapod_description/urdf/pexod.xacro (robot description, xacro)
@@ -7,5 +7,5 @@
   </xacro:if>
   <xacro:if value="${'relative' == path_generation}">
-    <xacro:property name="path_prefix" value="" />
+    <xacro:property name="path_prefix" value="./" />
   </xacro:if>
   <xacro:include filename="$(find hexapod_description)/urdf/modules/pexod.xacro" />
