Commit message: prepared for bringup

File: hexapod_description/urdf/mini_hexapod_visuals_collisions.xacro (robot description, xacro)
@@ -83,5 +83,5 @@
       <origin xyz="0 0 0" rpy="0 0 ${PI}"/>
       <geometry>
-        <mesh filename="${path_prefix + 'stl/third_link_v4.5.stl'}" scale="0.001 0.001 0.001"/>
+        <mesh filename="${path_prefix + 'stl/third_link_v5.stl'}" scale="0.001 0.001 0.001"/>
       </geometry>
       <material name="Red"/>

File: hexapod_description/urdf/modules/mini_hexapod.xacro (robot description, xacro)
@@ -30,8 +30,8 @@
   <xacro:property name="joint_dmp" value="0.25"/>
   <xacro:property name="joint_friction" value="0.183333333"/>
-  <xacro:include filename="$(find hexapod_description)/urdf/pexod_visuals_collisions.xacro" />
+  <xacro:include filename="$(find hexapod_description)/urdf/mini_hexapod_visuals_collisions.xacro" />
   <!-- Load xacro modules/parts of the robot -->
   <xacro:include filename="$(find hexapod_description)/urdf/modules/body.xacro" />
-  <xacro:include filename="$(find hexapod_description)/urdf/modules/leg_pexod.xacro" />
-  <xacro:include filename="$(find hexapod_description)/urdf/modules/legs_pexod.xacro" />
+  <xacro:include filename="$(find hexapod_description)/urdf/modules/leg_mini_hexapod.xacro" />
+  <xacro:include filename="$(find hexapod_description)/urdf/modules/legs_mini_hexapod.xacro" />
 </robot>
