Commit message: simplified mini hexa urdf to use with dart

File: hexapod_description/urdf/mini_hexapod.urdf (robot description, URDF)
Before this commit: robot mini_hexapod, 19 links, 18 joints
Links:
- link base_link: geometry collision box size=0.11 0.199 0.04; collision box size=0.24 0.119 0.04
- link leg_0_1: geometry collision box size=0.044 0.044 0.06; visual box size=0.044 0.044 0.06
- link leg_0_2: geometry collision box size=0.038 0.038 0.0835; visual box size=0.038 0.038 0.0835
- link leg_0_3: geometry collision box size=0.054 0.054 0.08; collision box size=0.054 0.065 0.054
- link leg_1_1: geometry collision box size=0.044 0.044 0.06; visual box size=0.044 0.044 0.06
- link leg_1_2: geometry collision box size=0.038 0.038 0.0835; visual box size=0.038 0.038 0.0835
- link leg_1_3: geometry collision box size=0.054 0.054 0.08; collision box size=0.054 0.065 0.054
- link leg_2_1: geometry collision box size=0.044 0.044 0.06; visual box size=0.044 0.044 0.06
- link leg_2_2: geometry collision box size=0.038 0.038 0.0835; visual box size=0.038 0.038 0.0835
- link leg_2_3: geometry collision box size=0.054 0.054 0.08; collision box size=0.054 0.065 0.054
- link leg_3_1: geometry collision box size=0.044 0.044 0.06; visual box size=0.044 0.044 0.06
- link leg_3_2: geometry collision box size=0.038 0.038 0.0835; visual box size=0.038 0.038 0.0835
- link leg_3_3: geometry collision box size=0.054 0.054 0.08; collision box size=0.054 0.065 0.054
- link leg_4_1: geometry collision box size=0.044 0.044 0.06; visual box size=0.044 0.044 0.06
- link leg_4_2: geometry collision box size=0.038 0.038 0.0835; visual box size=0.038 0.038 0.0835
- link leg_4_3: geometry collision box size=0.054 0.054 0.08; collision box size=0.054 0.065 0.054
- link leg_5_1: geometry collision box size=0.044 0.044 0.06; visual box size=0.044 0.044 0.06
- link leg_5_2: geometry collision box size=0.038 0.038 0.0835; visual box size=0.038 0.038 0.0835
- link leg_5_3: geometry collision box size=0.054 0.054 0.08; collision box size=0.054 0.065 0.054

File: hexapod_description/urdf/modules/mini_hexapod.xacro (robot description, xacro)
@@ -30,5 +30,5 @@
   <xacro:property name="joint_dmp" value="0.25"/>
   <xacro:property name="joint_friction" value="0.183333333"/>
-  <xacro:include filename="$(find hexapod_description)/urdf/mini_hexapod_visuals_collisions.xacro" />
+  <xacro:include filename="$(find hexapod_description)/urdf/mini_hexapod_visuals_collisions0.xacro" />
   <!-- Load xacro modules/parts of the robot -->
   <xacro:include filename="$(find hexapod_description)/urdf/modules/body.xacro" />

Commit message: fixed mini hexapod urdf for sim

File: hexapod_description/urdf/mini_hexapod.urdf (robot description, URDF)
Before this commit: robot mini_hexapod, 19 links, 18 joints
Links:
- link base_link: mass 1.031 -> 0.322; geometry collision box size=0.08625 0.095 0.035; collision box size=0.145 0.095 0.035
- link leg_0_1: mass 0.02 -> 0.01141; geometry collision box size=0.0345 0.0345 0.047; visual cylinder length=0.047 radius=0.01725
- link leg_0_2: mass 0.184 -> 0.04272; geometry collision box size=0.034 0.034 0.06; visual cylinder length=0.06 radius=0.017
- link leg_0_3: mass 0.04 -> 0.01457; geometry collision box size=0.0345 0.01 0.0345; collision box size=0.0345 0.0345 0.08
- link leg_1_1: mass 0.02 -> 0.01141; geometry collision box size=0.0345 0.0345 0.047; visual cylinder length=0.047 radius=0.01725
- link leg_1_2: mass 0.184 -> 0.04272; geometry collision box size=0.034 0.034 0.06; visual cylinder length=0.06 radius=0.017
- link leg_1_3: mass 0.04 -> 0.01457; geometry collision box size=0.0345 0.01 0.0345; collision box size=0.0345 0.0345 0.08
- link leg_2_1: mass 0.02 -> 0.01141; geometry collision box size=0.0345 0.0345 0.047; visual cylinder length=0.047 radius=0.01725
- link leg_2_2: mass 0.184 -> 0.04272; geometry collision box size=0.034 0.034 0.06; visual cylinder length=0.06 radius=0.017
- link leg_2_3: mass 0.04 -> 0.01457; geometry collision box size=0.0345 0.01 0.0345; collision box size=0.0345 0.0345 0.08
- link leg_3_1: mass 0.02 -> 0.01141; geometry collision box size=0.0345 0.0345 0.047; visual cylinder length=0.047 radius=0.01725
- link leg_3_2: mass 0.184 -> 0.04272; geometry collision box size=0.034 0.034 0.06; visual cylinder length=0.06 radius=0.017
- link leg_3_3: mass 0.04 -> 0.01457; geometry collision box size=0.0345 0.01 0.0345; collision box size=0.0345 0.0345 0.08
- link leg_4_1: mass 0.02 -> 0.01141; geometry collision box size=0.0345 0.0345 0.047; visual cylinder length=0.047 radius=0.01725
- link leg_4_2: mass 0.184 -> 0.04272; geometry collision box size=0.034 0.034 0.06; visual cylinder length=0.06 radius=0.017
- link leg_4_3: mass 0.04 -> 0.01457; geometry collision box size=0.0345 0.01 0.0345; collision box size=0.0345 0.0345 0.08
- link leg_5_1: mass 0.02 -> 0.01141; geometry collision box size=0.0345 0.0345 0.047; visual cylinder length=0.047 radius=0.01725
- link leg_5_2: mass 0.184 -> 0.04272; geometry collision box size=0.034 0.034 0.06; visual cylinder length=0.06 radius=0.017
- link leg_5_3: mass 0.04 -> 0.01457; geometry collision box size=0.0345 0.01 0.0345; collision box size=0.0345 0.0345 0.08
Joints:
- joint body_leg_0: origin xyz=-0.12 0.0595 0 rpy=0 0 0.3 -> xyz=-0.0725 0.0475 0 rpy=0 0 0.3
- joint body_leg_1: origin xyz=0 0.0995 0 rpy=0 0 0 -> xyz=0 0.0475 0 rpy=0 0 0
- joint body_leg_2: origin xyz=0.12 0.0595 0 rpy=0 0 -0.3 -> xyz=0.0725 0.0475 0 rpy=0 0 -0.3
- joint body_leg_3: origin xyz=0.12 -0.0595 0 rpy=0 0 3.44159265359 -> xyz=0.0725 -0.0475 0 rpy=0 0 3.44159265359
- joint body_leg_4: origin xyz=0 -0.0995 0 rpy=0 0 3.14159265359 -> xyz=0 -0.0475 0 rpy=0 0 3.14159265359
- joint body_leg_5: origin xyz=-0.12 -0.0595 0 rpy=0 0 2.84159265359 -> xyz=-0.0725 -0.0475 0 rpy=0 0 2.84159265359
- joint leg_0_1_2: origin xyz=0 0.06 0 rpy=0 0 0 -> xyz=0 0.047 0 rpy=0 0 0
- joint leg_0_2_3: origin xyz=0 0.0835 0 rpy=0 0 0 -> xyz=0 0.06 0 rpy=0 0 0
- joint leg_1_1_2: origin xyz=0 0.06 0 rpy=0 0 0 -> xyz=0 0.047 0 rpy=0 0 0
- joint leg_1_2_3: origin xyz=0 0.0835 0 rpy=0 0 0 -> xyz=0 0.06 0 rpy=0 0 0
- joint leg_2_1_2: origin xyz=0 0.06 0 rpy=0 0 0 -> xyz=0 0.047 0 rpy=0 0 0
- joint leg_2_2_3: origin xyz=0 0.0835 0 rpy=0 0 0 -> xyz=0 0.06 0 rpy=0 0 0
- joint leg_3_1_2: origin xyz=0 0.06 0 rpy=0 0 0 -> xyz=0 0.047 0 rpy=0 0 0
- joint leg_3_2_3: origin xyz=0 0.0835 0 rpy=0 0 0 -> xyz=0 0.06 0 rpy=0 0 0
- joint leg_4_1_2: origin xyz=0 0.06 0 rpy=0 0 0 -> xyz=0 0.047 0 rpy=0 0 0
- joint leg_4_2_3: origin xyz=0 0.0835 0 rpy=0 0 0 -> xyz=0 0.06 0 rpy=0 0 0
- joint leg_5_1_2: origin xyz=0 0.06 0 rpy=0 0 0 -> xyz=0 0.047 0 rpy=0 0 0
- joint leg_5_2_3: origin xyz=0 0.0835 0 rpy=0 0 0 -> xyz=0 0.06 0 rpy=0 0 0

File: hexapod_description/urdf/mini_hexapod_visuals_collisions0.xacro (robot description, xacro)
@@ -53,5 +53,5 @@
       <origin xyz="0 ${leg1_length/2} 0" rpy="${PI_2} 0 0"/>
         <geometry>
-          <box size="${leg1_width} ${leg1_width} ${leg1_length}"/>
+          <cylinder length="${leg1_length}" radius="${leg1_width/2.}"/>
         </geometry>
       <material name="Red"/>
@@ -67,7 +67,7 @@
     <visual>
       <origin xyz="0 ${leg2_length/2} 0" rpy="${PI_2} 0 0"/>
-        <geometry>
-          <box size="${leg2_width} ${leg2_width} ${leg2_length}"/>
-        </geometry>
+      <geometry>
+        <cylinder length="${leg2_length}" radius="${leg2_width/2.}"/>
+      </geometry>
       <material name="Blue"/>
     </visual>
@@ -82,7 +82,23 @@
     <visual>
       <origin xyz="0 ${leg3_length/2} 0" rpy="0 0 0"/>
+      <geometry>
+        <cylinder length="${leg3_width/2.}" radius="${leg3_length}"/>
+      </geometry>
+      <material name="Red"/>
+    </visual>
+    <visual>
+      <origin xyz="0 ${leg3_length-leg3_width/2} ${-(leg3_width+leg3_height-leg3_tip_radius)/2}"
+        rpy="0 0 0"/>
         <geometry>
-          <box size="${leg3_width} ${leg3_length} ${leg3_width}"/>
+          <cylinder length="${leg3_height-leg3_tip_radius}" radius="${leg3_width/2.}"/>
         </geometry>
+      <material name="Red"/>
+    </visual>
+    <visual>
+      <origin xyz="0 ${leg3_length-leg3_width/2} -${leg3_height}"
+        rpy="${PI_2} 0 0"/>
+            <geometry>
+                <sphere radius="${leg3_tip_radius}"/>
+            </geometry>
       <material name="Red"/>
     </visual>
